File: circuit/relay-001-20260624/relay-001-20260624.kicad_pcb (KiCad board)
At the start: 2 copper layers, 169 x 126.3 mm, 15 parts, among them J1 Conn_01x03_Pin, J10 Conn_01x02_Pin, J11 Conn_01x02_Pin, J12 Conn_01x02_Pin, J13 Conn_01x02_Pin, J14 Conn_01x02_Pin, J15 Conn_01x02_Pin, J2 Conn_02x05_Odd_Even, J3 Conn_02x08_Odd_Even, J4 Conn_02x09_Odd_Even, J5 Conn_01x02_Pin, J6 Conn_01x02_Pin, J7 Conn_01x02_Pin, J8 Conn_01x02_Pin, J9 Conn_01x02_Pin

Commit message: Update 供給基板のボード図を更新
Connections:
- J3 pad 13: +3.3V -> GND
- J3 pad 15: GND -> +3.3V
Routing:
- net Motor4_{PWM}: track 84.7 -> 87.4 mm
- net +3.3V: track 202.3 -> 201.3 mm
- net GND: vias 2634 -> 2609

Commit message: Update 供給基板を開いてちょっとシルクスクリーンを修正
Parts:
- J1: value Conn_01x03_Pin -> Dribbler_{Back}
- J11: value Conn_01x02_Pin -> Motor1
- J12: value Conn_01x02_Pin -> Motor2
- J13: value Conn_01x02_Pin -> Motor3
- J14: value Conn_01x02_Pin -> Motor4
- J2: value Conn_02x05_Odd_Even -> Kicker-Board
- J3: value Conn_02x08_Odd_Even -> MD-Board
- J4: value Conn_02x09_Odd_Even -> Main-Board
- J5, J8: value Conn_01x02_Pin -> Linesensor_{Power}
- J9: value Conn_01x02_Pin -> Linesensor_{UART}

Commit message: Update 供給基板のボード図を更新
Connections:
- J3 pad 1: BallCatch_{Back} -> Motor_{OUT4-2}
- J3 pad 10: Motor_{OUT2-2} -> Motor1_{PWM}
- J3 pad 11: Motor_{EN} -> Motor_{OUT2-1}
- J3 pad 12: Motor_{OUT2-1} -> Motor_{EN}
- J3 pad 13: GND -> Motor_{OUT1-2}
- J3 pad 14: Motor_{OUT1-2} -> GND
- J3 pad 15: +3.3V -> Motor_{OUT1-1}
- J3 pad 16: Motor_{OUT1-1} -> +3.3V
- J3 pad 2: Motor_{OUT4-2} -> BallCatch_{Back}
- J3 pad 3: Motor4_{PWM} -> Motor_{OUT4-1}
- J3 pad 4: Motor_{OUT4-1} -> Motor4_{PWM}
- J3 pad 5: Motor3_{PWM} -> Motor_{OUT3-2}
- J3 pad 6: Motor_{OUT3-2} -> Motor3_{PWM}
- J3 pad 7: Motor2_{PWM} -> Motor_{OUT3-1}
- J3 pad 8: Motor_{OUT3-1} -> Motor2_{PWM}
- J3 pad 9: Motor1_{PWM} -> Motor_{OUT2-2}
Routing:
- net Motor_{OUT3-2}: track 54.6 -> 108.5 mm
- net Motor_{OUT3-1}: track 46.9 -> 96.0 mm, vias 0 -> 6
- net Motor_{OUT2-1}: track 67.2 -> 108.2 mm
- net Motor_{OUT1-2}: track 137.0 -> 118.0 mm
- net Motor4_{PWM}: track 87.4 -> 104.9 mm, vias 4 -> 6
- net Dribbler_{Back}: track 76.8 -> 65.2 mm
- net Motor_{OUT1-1}: track 125.8 -> 136.1 mm
- net +3.3V: track 201.3 -> 208.9 mm, vias 6 -> 10
- net BallCatch_{Back}: track 88.2 -> 95.1 mm, vias 4 -> 5
- net Motor_{OUT2-2}: track 61.4 -> 67.2 mm
- net Motor_{OUT4-2}: track 99.4 -> 104.8 mm, vias 3 -> 9
- net Motor_{OUT4-1}: track 112.8 -> 115.1 mm, vias 3 -> 9
- net Motor1_{PWM}: track 104.0 -> 102.0 mm, vias 0 -> 2
- net BallCatch_{Front}: track 54.6 -> 53.0 mm
- net Motor_{EN}: track 100.6 -> 101.8 mm, vias 0 -> 1
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
Commit message: Update 供給基板のボード図の修正とDR完了、再DR求
Parts:
- J10: value Conn_01x02_Pin -> MD_{Power}
- J15: value Conn_01x02_Pin -> Voltmeter
- J3: value MD-Board -> MD_{Signal}
- J5: value Linesensor_{Power} -> Power_{5V}
- J6: value Conn_01x02_Pin -> Power_{VCC}
- J7: value Conn_01x02_Pin -> Power_{Logic}
- J8: value Linesensor_{Power} -> Line_{Power}
- J9: value Linesensor_{UART} -> Line_{UART}
- moved J1 160.6 mm to (-20.3, 1.93)
- moved J10 160.6 mm to (-14.0, 30.5)
- moved J11 160.6 mm to (-45.7, -28.0)
- moved J12 160.6 mm to (-47.4, 29.7)
- moved J13 160.6 mm to (45.7, 28.0)
- moved J14 160.6 mm to (47.5, -29.7)
- moved J15 160.6 mm to (-73.6, 6.80)
- moved J2 160.6 mm to (-5.08, -25.8)
- moved J3 160.6 mm to (0.43, 31.0)
- moved J4 160.6 mm to (55.2, -12.3)
- moved J5 160.6 mm to (-35.0, -11.0)
- moved J6 160.6 mm to (-35.0, 15.0)
- moved J7 160.6 mm to (-28.4, 2.00)
- moved J8 160.6 mm to (36.5, 19.5)
- moved J9 160.6 mm to (-41.3, 23.8)
Routing:
- net Motor_{OUT4-2}: track 104.8 -> 124.5 mm, vias 9 -> 20
- net Motor_{OUT3-1}: track 96.0 -> 113.2 mm, vias 6 -> 14
- net Motor_{OUT4-1}: track 115.1 -> 128.0 mm, vias 9 -> 19
- net Motor_{OUT1-1}: track 136.1 -> 123.2 mm, vias 6 -> 13
- net +5V_{Line}: track 100.5 -> 88.6 mm
- net Motor4_{PWM}: track 104.9 -> 112.2 mm
- net VCC: track 202.3 -> 209.2 mm, vias 6 -> 14
- net Motor_{OUT1-2}: track 118.0 -> 124.8 mm, vias 7 -> 12
- net Motor_{OUT3-2}: track 108.5 -> 114.0 mm
- net Motor3_{PWM}: track 111.5 -> 106.1 mm
- net Motor_{EN}: track 101.8 -> 96.5 mm
- net Motor2_{PWM}: track 106.9 -> 101.8 mm
- net Motor1_{PWM}: track 102.0 -> 97.8 mm
- net Motor_{OUT2-2}: track 67.2 -> 63.1 mm
- net BallCatch_{Back}: track 95.1 -> 97.6 mm
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Other:
- outline, holes or cut-outs redrawn
- board text added: "Relay-001"

Commit message: Update 供給基板の回路図PDF、PCBPDF、3Dモデル、発注ファイルを生成
Other:
- board text added: "+3.3V"
- board text added: "GND"
- board text added: "Sig"
