File: circuit/fpc_sub_neopixel-001-20260627/fpc_sub_neopixel-001-20260627.kicad_pcb (KiCad board)
At the start: 2 copper layers, 5.5 x 70 mm, 2 parts, among them J1 Conn_Sub, J2 Conn_NeoPixel

Commit message: Update NeoPixel-Sub
Parts:
- J1, J2: footprint @Thrive_footprint_fpc_sub_neopixel:AFC01-S10FCA-00 -> @Thrive_footprint_fpc_sub_neopixel:AFC01-S12FCA-00
Connections:
- J2 pad 1: Net-(J1-Pin_10) -> Net-(J1-Pin_12)
- J2 pad 10: Net-(J1-Pin_1) -> Net-(J1-Pin_3)
- J2 pad 2: Net-(J1-Pin_9) -> Net-(J1-Pin_11)
- J2 pad 3: Net-(J1-Pin_8) -> Net-(J1-Pin_10)
- J2 pad 4: Net-(J1-Pin_7) -> Net-(J1-Pin_9)
- J2 pad 5: Net-(J1-Pin_6) -> Net-(J1-Pin_8)
- J2 pad 6: Net-(J1-Pin_5) -> Net-(J1-Pin_7)
- J2 pad 7: Net-(J1-Pin_4) -> Net-(J1-Pin_6)
- J2 pad 8: Net-(J1-Pin_3) -> Net-(J1-Pin_5)
- J2 pad 9: Net-(J1-Pin_2) -> Net-(J1-Pin_4)
Routing:
- net Net-(J1-Pin_12): track 0.00 -> 73.0 mm
- net Net-(J1-Pin_11): track 0.00 -> 73.0 mm
Other:
- board size 5.5 x 70 mm -> 6.5 x 70 mm
