File: circuit/fpc_sub_neopixel-001-20260627/fpc_sub_neopixel-001-20260627.kicad_sch (KiCad schematic)
At the start: 2 parts, among them J1 Conn_Sub, J2 Conn_NeoPixel

Commit message: Update NeoPixel-Sub
Parts:
- removed J1: Conn_Sub, @Thrive_footprint_fpc_sub_neopixel:AFC01-S10FCA-00, symbol Connector:Conn_01x10_Pin
- removed J2: Conn_NeoPixel, @Thrive_footprint_fpc_sub_neopixel:AFC01-S10FCA-00, symbol Connector:Conn_01x10_Pin
- added J1: Conn_Sub, @Thrive_footprint_fpc_sub_neopixel:AFC01-S12FCA-00, symbol Connector:Conn_01x12_Pin
- added J2: Conn_NeoPixel, @Thrive_footprint_fpc_sub_neopixel:AFC01-S12FCA-00, symbol Connector:Conn_01x12_Pin
Connections:
- new net: J1.1 (Pin_1), J2.12 (Pin_12)
- new net: J1.10 (Pin_10), J2.3 (Pin_3)
- new net: J1.11 (Pin_11), J2.2 (Pin_2)
- new net: J1.12 (Pin_12), J2.1 (Pin_1)
- new net: J1.2 (Pin_2), J2.11 (Pin_11)
- new net: J1.3 (Pin_3), J2.10 (Pin_10)
- new net: J1.4 (Pin_4), J2.9 (Pin_9)
- new net: J1.5 (Pin_5), J2.8 (Pin_8)
- new net: J1.6 (Pin_6), J2.7 (Pin_7)
- new net: J1.7 (Pin_7), J2.6 (Pin_6)
- new net: J1.8 (Pin_8), J2.5 (Pin_5)
- new net: J1.9 (Pin_9), J2.4 (Pin_4)
Changed lines of the file:
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@@
+	(wire
+		(pts
+			(xy 38.1 55.88) (xy 43.18 55.88)
+		)
+		(stroke
+			(width 0)
+			(type default)
+		)
+	)
 	(wire
 		(pts
@@
 	(wire
 		(pts
+			(xy 38.1 53.34) (xy 43.18 53.34)
+		)
+		(stroke
+			(width 0)
+			(type default)
+		)
+	)
+	(wire
+		(pts
 			(xy 43.18 40.64) (xy 38.1 40.64)
 		)
@@
 	)
 	(symbol
-		(lib_id "Connector:Conn_01x10_Pin")
-		(at 33.02 38.1 0)
+		(lib_id "Connector:Conn_01x12_Pin")
+		(at 33.02 40.64 0)
 		(unit 1)
 		(body_style 1)
@@
 			)
 		)
-		(property "Footprint" "@Thrive_footprint_fpc_sub_neopixel:AFC01-S10FCA-00"
-			(at 33.02 38.1 0)
+		(property "Footprint" "@Thrive_footprint_fpc_sub_neopixel:AFC01-S12FCA-00"
+			(at 33.02 40.64 0)
 			(hide yes)
 			(show_name no)
@@
 		)
 		(property "Datasheet" ""
-			(at 33.02 38.1 0)
-			(hide yes)
-			(show_name no)
-			(do_not_autoplace no)
-			(effects
-				(font
-					(size 1.27 1.27)
-				)
-			)
-		)
-		(property "Description" "Generic connector, single row, 01x10, script generated"
-			(at 33.02 38.1 0)
-			(hide yes)
-			(show_name no)
-			(do_not_autoplace no)
-			(effects
-				(font
-					(size 1.27 1.27)
-				)
-			)
+			(at 33.02 40.64 0)
+			(hide yes)
+			(show_name no)
+			(do_not_autoplace no)
+			(effects
+				(font
+					(size 1.27 1.27)
+				)
+			)
+		)
+		(property "Description" "Generic connector, single row, 01x12, script generated"
+			(at 33.02 40.64 0)
+			(hide yes)
+			(show_name no)
+			(do_not_autoplace no)
+			(effects
+				(font
+					(size 1.27 1.27)
+				)
+			)
+		)
+		(pin "1"
+		)
+		(pin "12"
+		)
+		(pin "3"
+		)
+		(pin "6"
 		)
 		(pin "4"
 		)
-		(pin "3"
-		)
-		(pin "6"
-		)
 		(pin "5"
 		)
+		(pin "8"
+		)
+		(pin "10"
+		)
+		(pin "7"
+		)
 		(pin "9"
 		)
-		(pin "1"
-		)
 		(pin "2"
 		)
-		(pin "7"
-		)
-		(pin "8"
-		)
-		(pin "10"
+		(pin "11"
 		)
 		(instances
@@
 	)
 	(symbol
-		(lib_id "Connector:Conn_01x10_Pin")
-		(at 48.26 40.64 180)
+		(lib_id "Connector:Conn_01x12_Pin")
+		(at 48.26 43.18 180)
 		(unit 1)
 		(body_style 1)
@@
 		(dnp no)
 		(property "Reference" "J2"
-			(at 47.625 55.88 0)
+			(at 47.625 60.96 0)
 			(show_name no)
 			(do_not_autoplace no)
@@
 		)
 		(property "Value" "Conn_NeoPixel"
-			(at 47.625 53.34 0)
-			(show_name no)
-			(do_not_autoplace no)
-			(effects
-				(font
-					(size 1.27 1.27)
-				)
-			)
-		)
-		(property "Footprint" "@Thrive_footprint_fpc_sub_neopixel:AFC01-S10FCA-00"
-			(at 48.26 40.64 0)
+			(at 47.625 58.42 0)
+			(show_name no)
+			(do_not_autoplace no)
+			(effects
+				(font
+					(size 1.27 1.27)
+				)
+			)
+		)
+		(property "Footprint" "@Thrive_footprint_fpc_sub_neopixel:AFC01-S12FCA-00"
+			(at 48.26 43.18 0)
 			(hide yes)
 			(show_name no)
@@
 		)
 		(property "Datasheet" ""
-			(at 48.26 40.64 0)
-			(hide yes)
-			(show_name no)
-			(do_not_autoplace no)
-			(effects
-				(font
-					(size 1.27 1.27)
-				)
-			)
-		)
-		(property "Description" "Generic connector, single row, 01x10, script generated"
-			(at 48.26 40.64 0)
-			(hide yes)
-			(show_name no)
-			(do_not_autoplace no)
-			(effects
-				(font
-					(size 1.27 1.27)
-				)
-			)
+			(at 48.26 43.18 0)
+			(hide yes)
+			(show_name no)
+			(do_not_autoplace no)
+			(effects
+				(font
+					(size 1.27 1.27)
+				)
+			)
+		)
+		(property "Description" "Generic connector, single row, 01x12, script generated"
+			(at 48.26 43.18 0)
+			(hide yes)
+			(show_name no)
+			(do_not_autoplace no)
+			(effects
+				(font
+					(size 1.27 1.27)
+				)
+			)
+		)
+		(pin "1"
+		)
+		(pin "12"
+		)
+		(pin "3"
+		)
+		(pin "6"
 		)
 		(pin "4"
 		)
-		(pin "3"
-		)
-		(pin "6"
-		)
 		(pin "5"
 		)
+		(pin "8"
+		)
+		(pin "10"
+		)
+		(pin "7"
+		)
 		(pin "9"
 		)
-		(pin "1"
-		)
 		(pin "2"
 		)
-		(pin "7"
-		)
-		(pin "8"
-		)
-		(pin "10"
+		(pin "11"
 		)
 		(instances
