File: circuit/power-001-20260513/power-001-20260513.kicad_pcb (KiCad board)
At the start: 2 copper layers, 68.4 x 46.4 mm, 46 parts, among them J2 +5V_{Line}, J3 Power, J4 Logic, J5 Sub_{Power}, J6 Sub_{Signal}, Q1 BSS138, Q2 PMOS, U1 OKL-T/6-W12N-C, U2 OKL-T/6-W12N-C, U3 AZ1084-3.3, U4 BP5293-33, U5 PIC12F683-xSN

Commit message: Update コートヤード要件を追加した
Parts:
- added F1: 10A, @Thrive_footprint_power:MF61NR_FUC-04, F.Cu at (120.5, 75.0)
- added J1: VIN, @Thrive_footprint_power:Conn_01x02_Wire_Only, B.Cu at (120.5, 75.0)
- added SW1: SW_SPDT, @Thrive_footprint_power:2MS1-T1-B4-M2-Q-E, F.Cu at (88.7, 68.3)
- added SW2: SW_SPDT, @Thrive_footprint_power:2MS1-T1-B4-M2-Q-E, F.Cu at (97.7, 68.3)
- added SW3: SW_SPDT, @Thrive_footprint_power:2MS1-T1-B4-M2-Q-E, F.Cu at (106.7, 68.3)
- added SW4: Locker_SW, @Thrive_footprint_power:DS-850K-S-ON-K, F.Cu at (97.9, 81.8)
- added TP1: TP_{+5V-Line}, TestPoint:TestPoint_Loop_D1.80mm_Drill1.0mm_Beaded, F.Cu at (146.6, 63.1)
- added TP2: TP_{+5V-Line}, TestPoint:TestPoint_Loop_D1.80mm_Drill1.0mm_Beaded, F.Cu at (146.6, 67.7)
- added TP3: TP_{+5V}, TestPoint:TestPoint_Loop_D1.80mm_Drill1.0mm_Beaded, F.Cu at (146.6, 72.4)
- added TP4: TP_{+3.3V}, TestPoint:TestPoint_Loop_D1.80mm_Drill1.0mm_Beaded, F.Cu at (146.6, 77.0)
- added TP5: TP_{GND}, TestPoint:TestPoint_Loop_D1.80mm_Drill1.0mm_Beaded, F.Cu at (146.6, 81.7)
- moved U4 93.4 mm to (158.1, 66.9)
- moved BZ1 73.1 mm to (135.7, 99.1)
- moved U1 62.2 mm to (134.2, 66.3)
- moved U2 59.2 mm to (136.5, 84.2)
- moved D1 57.8 mm to (151.7, 101.7)
- moved Q1 57.8 mm to (147.0, 102.8)
- moved Q2 57.7 mm to (151.2, 88.2)
- moved U3 57.7 mm to (151.2, 96.4)
- moved C11 55.5 mm to (163.1, 94.5)
- moved C12 55.5 mm to (163.1, 97.6)
- moved C2 55.5 mm to (158.7, 85.5)
- moved C3 55.5 mm to (158.7, 88.5)
- moved C6 55.5 mm to (158.7, 94.5)
- moved C7 55.5 mm to (158.7, 97.6)
- moved C8 55.5 mm to (163.1, 85.5)
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Connections:
- J4 pad 1: +5V -> +3.3V
- J4 pad 2: +3.3V -> +5V
Other:
- outline, holes or cut-outs redrawn

Commit message: Update 電源基板に部品を軽く配置した（違法建築あり）
Parts:
- BZ1, Q1, Q2, U4: moved to B.Cu
- moved U1 81.1 mm to (60.0, 99.0), turned to 180 degrees
- moved U3 80.3 mm to (72.0, 83.0)
- moved Q2 67.0 mm to (84.7, 96.7), turned to 180 degrees
- moved U2 64.9 mm to (75.3, 106.1)
- moved Q1 53.7 mm to (94.1, 93.5)
- moved U4 53.6 mm to (110.8, 92.2), turned to -90 degrees
- moved U5 37.0 mm to (132.8, 126.7)
- moved BZ1 32.3 mm to (108.0, 82.5), turned to -90 degrees
- moved SW3 18.5 mm to (100.0, 85.5)
- moved C10 17.7 mm to (159.0, 108.8)
- moved C12 17.7 mm to (159.0, 114.8)
- moved C3 17.7 mm to (154.5, 105.8)
- moved C4 17.7 mm to (154.5, 108.8)
- moved C7 17.7 mm to (154.5, 114.8)
- moved C9 17.7 mm to (159.0, 105.8)
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
Commit message: Update ちょっと電源基板を修正
Parts:
- added J7: ICSP_{PIC12F683}, Connector_PinHeader_2.54mm:PinHeader_1x05_P2.54mm_Vertical, F.Cu at (152.2, 108.8)
- added R21: 10k, Resistor_SMD:R_0805_2012Metric, F.Cu at (143.0, 110.7)
- D1: footprint Capacitor_SMD:C_0603_1608Metric -> LED_SMD:LED_0603_1608Metric
- R16: value 1.2k -> 330
- R17: value 100 -> 1.2k
- R18: value 10k -> 100
- R20: value 330 -> 10k
- moved R6 26.2 mm to (134.2, 107.7)
- moved R7 26.2 mm to (134.2, 110.7)
- moved R11 22.1 mm to (138.6, 101.8)
- moved R12 22.1 mm to (138.6, 104.8)
- moved R13 22.1 mm to (138.6, 107.7)
- moved R14 22.1 mm to (138.6, 110.7)
- moved R16 19.0 mm to (143.0, 95.9)
- moved R17 19.0 mm to (143.0, 98.9)
- moved R18 19.0 mm to (143.0, 101.8)
- moved R19 19.0 mm to (143.0, 104.8)
- moved R20 19.0 mm to (143.0, 107.7)
- moved R15 14.5 mm to (143.0, 93.0)
- moved TP1 14.4 mm to (147.6, 93.8)
- moved TP2 14.4 mm to (147.6, 98.5)
- moved TP3 14.4 mm to (147.6, 103.1)
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Connections:
- net Prot-Vraw renamed ICSPDAT
- R16 pad 1: Net-(BZ1-+) -> Prot-LED
- R16 pad 2: Prot-Buzzer -> Net-(D1-A)
- R17 pad 1: Prot-CTRL -> Net-(BZ1-+)
- R17 pad 2: Net-(Q1-G) -> Prot-Buzzer
- R18 pad 1: GND -> ICSPCLK
- R19 pad 1: Net-(Q1-D) -> GND
- R19 pad 2: VCC -> Net-(Q1-G)
- R20 pad 1: Net-(D1-A) -> Net-(Q1-D)
- R20 pad 2: Prot-LED -> VCC
- U5 pad 3: unconnected-(U5-GP4-Pad3) -> Prot-LED
- U5 pad 4: Prot-LED -> MCLR
- U5 pad 6: Prot-CTRL -> ICSPCLK
