File: circuit/power-001-20260513/power-001-20260513.kicad_sch (KiCad schematic)
At the start: 49 parts, among them J1 VIN, J2 +5V_{Line}, J3 Power, J4 Logic, J5 Sub_{Power}, J6 Sub_{Signal}, J7 ICSP_{PIC12F683}, J8 ESC, Q1 BSS138, Q2 PMOS, SW1 SW_SPDT, SW2 SW_SPDT, SW4 Locker_SW, U1 OKL-T/6-W12N-C, U2 OKL-T/6-W12N-C, U3 AZ1084-3.3, U5 PIC12F683-xSN, U6 LM1117MP-3.3

Commit message: Update 電源基板のDRを受けてR10を修正
Parts:
- R10: value 1.5k -> 1k
Changed lines of the file:
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@@
 			)
 		)
-		(property "Value" "1.5k"
+		(property "Value" "1k"
 			(at 113.03 85.09 90)
 			(show_name no)

Commit message: Update 電源基板のシルクを整えた
Parts:
- Q2: value PMOS -> TJ60S04M3L
- U5: value PIC12F683-xSN -> PIC12F683
Changed lines of the file:
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@@
 			)
 		)
-		(property "Value" "PIC12F683-xSN"
+		(property "Value" "PIC12F683"
 			(at 209.5356 26.67 0)
 			(show_name no)
@@
 			)
 		)
-		(property "Value" "PMOS"
+		(property "Value" "TJ60S04M3L"
 			(at 251.46 49.53 90)
 			(show_name no)

Commit message: Update 電源基板の1000μF→470μF
Parts:
- C1: value 1000μ -> 470μ; footprint Capacitor_THT:CP_Radial_D10.0mm_P5.00mm -> Capacitor_THT:CP_Radial_D8.0mm_P3.50mm
Changed lines of the file:
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@@
 			)
 		)
-		(property "Value" "1000μ"
+		(property "Value" "470μ"
 			(at 41.91 76.1999 0)
 			(show_name no)
@@
 			)
 		)
-		(property "Footprint" "Capacitor_THT:CP_Radial_D10.0mm_P5.00mm"
+		(property "Footprint" "Capacitor_THT:CP_Radial_D8.0mm_P3.50mm"
 			(at 39.0652 78.74 0)
 			(hide yes)
