File: circuit/sub-001-20260515/sub-001-20260515.kicad_pcb (KiCad board)
At the start: 2 copper layers, 114.3 x 107 mm, 148 parts, among them J1 Conn_NeoPixel, J2 Conn_SW_TGL, J3 Conn_Power, J4 Conn_Main, Q1 BSS138, Q2 BSS138, Q3 BSS138, Q4 BSS138, Q5 BSS138, Q6 BSS138, Q7 BSS138, Q8 BSS138, U11 LM1117GS-3.3, U12 NE555DR, U13 NE555DR, U14 LM1117GS-3.3, U15 LM1117GS-3.3, U18 NE555DR, U19 NE555DR, U2 LM1117GS-3.3, U20 TSSP58038, U21 TSSP58038, U22 NE555DR, U23 NE555DR, U24 TSSP58038, U25 TSSP58038, U26 HC-SR04, U27 HC-SR04, U28 HC-SR04, U29 HC-SR04, U4 NE555DR, U5 NE555DR, U7 LM1117GS-3.3, U9 LM1117MP-3.3

Commit message: Update サブ基板のIR周りを完成させた
Parts:
- J2, J3: moved to B.Cu
- moved U25 322.8 mm to (-35.3, -38.9), turned to -135 degrees
- moved C48 317.7 mm to (-35.9, -33.0), turned to 90 degrees
- moved R46 312.5 mm to (-33.9, -34.9), turned to -90 degrees
- moved R39 311.5 mm to (-35.9, -29.5), turned to 90 degrees
- moved R37 307.8 mm to (-33.9, -30.4), turned to -90 degrees
- moved R40 307.1 mm to (-26.4, -38.6), turned to -90 degrees
- moved R38 306.2 mm to (-26.4, -42.2), turned to -90 degrees
- moved C40 305.3 mm to (-20.4, -43.9), turned to 90 degrees
- moved C39 304.6 mm to (-28.8, -29.7)
- moved R44 304.4 mm to (-27.2, -35.3)
- moved R43 304.3 mm to (-33.1, -18.6), turned to 90 degrees
- moved R33 302.0 mm to (-31.7, -30.4), turned to -90 degrees
- moved R42 301.8 mm to (-27.1, -33.0), turned to 180 degrees
- moved C45 301.3 mm to (-26.8, -22.9), turned to 90 degrees
- moved C46 300.9 mm to (-17.9, -37.5)
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Routing:
- net +5V: track 0.00 -> 161.4 mm, vias 0 -> 16
- net Net-(Q1-G): track 0.00 -> 14.1 mm
- net Net-(Q3-G): track 0.00 -> 14.0 mm
- net Net-(Q7-G): track 0.00 -> 13.8 mm
- net Net-(U18-THRES): track 0.00 -> 10.4 mm
- net Net-(U22-THRES): track 0.00 -> 10.4 mm
- net Net-(U12-THRES): track 0.00 -> 10.4 mm
- net Net-(U4-THRES): track 0.00 -> 10.4 mm
- net Net-(U23-THRES): track 0.00 -> 9.68 mm
- net Net-(U13-THRES): track 0.00 -> 9.68 mm
- net Net-(U5-THRES): track 0.00 -> 9.68 mm
- net Net-(U19-THRES): track 0.00 -> 9.68 mm
- net Net-(U18-OUT): track 0.00 -> 7.51 mm, vias 0 -> 2
- net Net-(Q5-G): track 0.00 -> 7.22 mm
- net Net-(Q8-G): track 0.00 -> 7.16 mm
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
Commit message: Update サブ基板のPCBを進めた
Parts:
- moved J3 133.2 mm to (-28.4, -13.7), turned to 90 degrees
- moved R41 2.22 mm to (-32.9, -18.6)
- moved R43 2.22 mm to (-35.3, -18.6)
Routing:
- net Net-(U22-OUT): track 2.72 -> 3.91 mm
- net Net-(Q7-G): track 13.8 -> 12.9 mm
- added copper zone on F.Cu, net +5V
- added copper zone on B.Cu, net GND

Commit message: Update サブ基板のコンポーネントを仮配置した
Parts:
- moved D4 244.2 mm to (-49.0, -21.9)
- moved D3 243.0 mm to (-49.0, -19.4)
- moved R16 234.5 mm to (-44.0, -21.9), turned to 180 degrees
- moved R15 233.1 mm to (-44.0, -19.0), turned to 180 degrees
- moved U8 173.6 mm to (-32.2, -1.17), turned to 180 degrees
- moved J1 158.3 mm to (0.00, -25.0)
- moved J4 154.7 mm to (-14.0, -25.0)
- moved U6 135.2 mm to (10.8, 32.2), turned to -90 degrees
- moved U14 132.3 mm to (-48.0, 0.00), turned to 90 degrees
- moved U9 126.2 mm to (-42.0, -12.0), turned to 180 degrees
- moved U10 124.3 mm to (25.2, -2.83)
- moved U1 119.6 mm to (-2.83, -32.2), turned to 90 degrees
- moved U11 98.3 mm to (0.00, 48.0), turned to 180 degrees
- moved U3 95.5 mm to (32.2, -2.83)
- moved U2 86.6 mm to (0.00, -48.0)
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Routing:
- net +5V: track 161.4 -> 370.8 mm, vias 16 -> 63
- net GND: track 3.37 -> 79.1 mm, vias 0 -> 59
- net Net-(U19-OUT): track 0.00 -> 5.93 mm
- net Net-(U23-OUT): track 0.00 -> 5.68 mm
- net Net-(U18-DISCH): track 5.14 -> 9.72 mm
- net Net-(U18-CONT): track 0.00 -> 4.15 mm, vias 0 -> 2
- net Net-(U18-OUT): track 7.51 -> 11.1 mm, vias 2 -> 0
- net Net-(D7-K): track 0.00 -> 2.43 mm
- net Net-(U18-THRES): track 10.4 -> 12.8 mm, vias 0 -> 2
- added copper zone on F.Cu, net GND
- removed copper zone on F.Cu, net +5V
