File: circuit/sub-001-20260515/sub-001-20260515.kicad_pcb (KiCad board)
At the start: 2 copper layers, 114.3 x 107 mm, 147 parts, among them J1 Conn_NeoPixel, J2 Conn_01x02_Socket, J3 Conn_Power, J4 Conn_Main, Q1 BSS138, Q2 BSS138, Q3 BSS138, Q4 BSS138, Q5 BSS138, Q6 BSS138, Q7 BSS138, Q8 BSS138, U11 LM1117GS-3.3, U12 NE555DR, U13 NE555DR, U14 LM1117GS-3.3, U15 LM1117GS-3.3, U18 NE555DR, U19 NE555DR, U2 LM1117GS-3.3, U20 TSSP58038, U21 TSSP58038, U22 NE555DR, U23 NE555DR, U24 TSSP58038, U25 TSSP58038, U26 HC-SR04, U27 HC-SR04, U28 HC-SR04, U29 HC-SR04, U4 NE555DR, U5 NE555DR, U7 LM1117GS-3.3, U9 LM1117MP-3.3

Commit message: Update サブ基板にビアを打ちまくった
Routing:
- net GND: vias 167 -> 2610
