File: circuit/line-001-20260628/line-001-20260628.kicad_pcb (KiCad board)
At the start: 2 copper layers, 217 parts, among them J1 Relay_{Power}, J2 Conn_{Signal}, J3 ICSP_{Arduino}, P1 USB-typeC, Q1 NJL7502L, Q10 NJL7502L, Q11 NJL7502L, Q12 NJL7502L, Q13 NJL7502L, Q14 NJL7502L, Q15 NJL7502L, Q16 NJL7502L, Q17 NJL7502L, Q18 NJL7502L, Q19 NJL7502L, Q2 NJL7502L, Q20 NJL7502L, Q21 NJL7502L, Q22 NJL7502L, Q23 NJL7502L, Q24 NJL7502L, Q25 NJL7502L, Q26 NJL7502L, Q27 NJL7502L, Q28 NJL7502L, Q29 NJL7502L, Q3 NJL7502L, Q30 NJL7502L, Q31 NJL7502L, Q32 NJL7502L, Q33 NJL7502L, Q34 NJL7502L, Q35 NJL7502L, Q36 NJL7502L, Q4 NJL7502L, Q5 NJL7502L, Q6 NJL7502L, Q7 NJL7502L, Q8 NJL7502L, Q9 NJL7502L, SW1 RESET, U1 LM339DR, U10 LM339DR, U11 LM339DR, U12 LM339DR, U13 LM339DR, U14 LM339DR, U15 LM339DR, U16 LM339DR, U17 ATmega2560-16A, U18 CH340G, U2 LM339DR, U3 LM339DR, U4 LM339DR, U5 LM339DR, U6 LM339DR, U7 LM339DR, U8 LM339DR, U9 LM339DR, Y1 16MHz, Y2 12MHz

Commit message: Update ラインセンサのボード図作成を開始した
Parts:
- added REF**: MountingHole_3.2mm_M3, MountingHole:MountingHole_3.2mm_M3, F.Cu at (67.1, -19.7)
- added REF**: MountingHole_3.2mm_M3, MountingHole:MountingHole_3.2mm_M3, F.Cu at (-67.1, -19.7)
- added REF**: MountingHole_3.2mm_M3, MountingHole:MountingHole_3.2mm_M3, F.Cu at (-67.1, 19.7)
- added REF**: MountingHole_3.2mm_M3, MountingHole:MountingHole_3.2mm_M3, F.Cu at (67.1, 19.7)
- D1, D10, D11, D12, D13, D14, D15, D16, D17, D18, D19, D2, D20, D21, D22, D23, D24, D25, D26, D27, D28, D29, D3, D30, D31, D32, D33, D34, D35, D36, D4, D5, D6, D7, D8, D9, Q1, Q10, Q11, Q12, Q13, Q14, Q15, Q16, Q17, Q18, Q19, Q2, Q20, Q21, Q22, Q23, Q24, Q25, Q26, Q27, Q28, Q29, Q3, Q30, Q31, Q32, Q33, Q34, Q35, Q36, Q4, Q5, Q6, Q7, Q8, Q9: moved to B.Cu
- moved Q30 188.0 mm to (-31.9, -47.8), turned to -56.25 degrees
- moved Q29 184.3 mm to (-40.7, -40.7), turned to -45 degrees
- moved Q28 179.5 mm to (-47.8, -31.9), turned to -33.75 degrees
- moved Q27 173.9 mm to (-53.1, -22.0), turned to -22.5 degrees
- moved Q31 168.4 mm to (-22.0, -53.1), turned to -67.5 degrees
- moved Q32 168.1 mm to (-11.2, -56.4), turned to -78.75 degrees
- moved Q26 167.5 mm to (-56.4, -11.2), turned to -11.25 degrees
- moved Q24 162.6 mm to (-56.4, 11.2), turned to 11.25 degrees
- moved Q25 160.4 mm to (-57.5, 0.00)
- moved Q23 151.6 mm to (-53.1, 22.0), turned to 22.5 degrees
- moved D30 148.4 mm to (-35.6, -53.3), turned to -56.25 degrees
- moved D29 144.3 mm to (-45.3, -45.3), turned to -45 degrees
- moved Q1 143.8 mm to (0.00, -57.5), turned to -90 degrees
- moved Q2 143.2 mm to (11.2, -56.4), turned to -101.25 degrees
- moved Q3 141.6 mm to (22.0, -53.1), turned to -112.5 degrees
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Other:
- board outline added: 162.9 x 133.7 mm

Commit message: Update ラインセンサ基板を更新
Parts:
- removed P1: USB-typeC, Connector_USB:USB_C_Receptacle_GCT_USB4105-xx-A_16P_TopMnt_Horizontal
- removed R83: 22, Resistor_SMD:R_0805_2012Metric
- removed the REF** at (67.1, -19.7)
- removed the REF** at (-67.1, -19.7)
- removed the REF** at (-67.1, 19.7)
- removed the REF** at (67.1, 19.7)
- added D39: LED_{USB}, LED_SMD:LED_0603_1608Metric, F.Cu at (220.1, 153.3)
- added J4: USB_C_Receptacle_USB2.0_16P, Connector_USB:USB_C_Receptacle_HCTL_HC-TYPE-C-16P-01A, F.Cu at (81.1, 10.6)
- added R86: 5.1k, Resistor_SMD:R_0805_2012Metric, F.Cu at (270.9, 91.6)
- added REF**: MountingHole_3.2mm_M3, MountingHole:MountingHole_3.2mm_M3, F.Cu at (6.50, -31.9)
- added REF**: MountingHole_3.2mm_M3, MountingHole:MountingHole_3.2mm_M3, F.Cu at (67.1, 19.7)
- added REF**: MountingHole_3.2mm_M3, MountingHole:MountingHole_3.2mm_M3, F.Cu at (-6.50, -31.9)
- added REF**: MountingHole_3.2mm_M3, MountingHole:MountingHole_3.2mm_M3, F.Cu at (-67.1, -19.7)
- added REF**: MountingHole_3.2mm_M3, MountingHole:MountingHole_3.2mm_M3, F.Cu at (67.1, -19.7)
- added REF**: MountingHole_3.2mm_M3, MountingHole:MountingHole_3.2mm_M3, F.Cu at (-67.1, 19.7)
- D1, D10, D11, D12, D13, D14, D15, D16, D17, D18, D19, D2, D20, D21, D22, D23, D24, D25, D26, D27, D28, D29, D3, D30, D31, D32, D33, D34, D35, D36, D4, D5, D6, D7, D8, D9, Q1, Q10, Q11, Q12, Q13, Q14, Q15, Q16, Q17, Q18, Q19, Q2, Q20, Q21, Q22, Q23, Q24, Q25, Q26, Q27, Q28, Q29, Q3, Q30, Q31, Q32, Q33, Q34, Q35, Q36, Q4, Q5, Q6, Q7, Q8, Q9: moved to F.Cu
- R82: value 22 -> 330
- moved Q29 344.9 mm to (260.8, 126.8), turned to 0 degrees
- moved Q28 344.6 mm to (260.8, 121.4), turned to 0 degrees
- moved Q30 343.7 mm to (260.8, 132.3), turned to 0 degrees
- moved Q27 342.9 mm to (260.8, 115.9), turned to 0 degrees
- moved Q26 339.8 mm to (260.8, 110.5), turned to 0 degrees
- moved Q25 335.2 mm to (260.8, 105.0)
- moved Q24 334.5 mm to (255.4, 132.3), turned to 0 degrees
- moved Q31 328.8 mm to (266.3, 105.0), turned to 0 degrees
- moved Q23 325.8 mm to (255.4, 126.8), turned to 0 degrees
- moved Q32 323.8 mm to (266.3, 110.5), turned to 0 degrees
- moved Q22 316.1 mm to (255.4, 121.4), turned to 0 degrees
- moved D28 307.2 mm to (227.7, 88.6), turned to 0 degrees
- moved D29 306.6 mm to (227.7, 94.1), turned to 0 degrees
- moved D27 306.5 mm to (227.7, 83.2), turned to 0 degrees
- moved Q21 305.5 mm to (255.4, 115.9), turned to 0 degrees
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Connections:
- R82 pad 1: Net-(P1-D-) -> VBUS
- R82 pad 2: D- -> Net-(D39-A)
Other:
- outline, holes or cut-outs redrawn
- board text added: "ここら辺にUARTの XHコネクタ配置"

Commit message: Update ラインセンサ基板の回路図とボード図を更新
Parts:
- removed D39: LED_{USB}, LED_SMD:LED_0603_1608Metric
- removed R79, R80: 330, Resistor_SMD:R_0805_2012Metric
- removed R81: 1M, Resistor_SMD:R_0805_2012Metric
- removed R84, R86: 5.1k, Resistor_SMD:R_0805_2012Metric
- removed R85: 10k, Resistor_SMD:R_0805_2012Metric
- removed the REF** at (6.50, -31.9)
- removed the REF** at (67.1, 19.7)
- removed the REF** at (-6.50, -31.9)
- removed the REF** at (-67.1, -19.7)
- removed the REF** at (67.1, -19.7)
- removed the REF** at (-67.1, 19.7)
- added D42: LED, LED_THT:LED_D3.0mm, B.Cu at (-69.0, -6.04)
- added D43: LED, LED_THT:LED_D3.0mm, B.Cu at (-69.0, 6.04)
- added D47: D40, LED_SMD:LED_0603_1608Metric, F.Cu at (113.2, 80.3)
- added D48: D41, LED_SMD:LED_0603_1608Metric, F.Cu at (113.2, 82.8)
- added D49: ~, Package_TO_SOT_SMD:TSOT-23, F.Cu at (84.2, 99.8)
- added D50: LED_{USB}, LED_SMD:LED_0603_1608Metric, F.Cu at (113.2, 85.4)
- added Q37: NJL7502L, @Thrive_footprint_kicker:NJL7502L, B.Cu at (73.7, -6.45)
- added Q38: NJL7502L, @Thrive_footprint_kicker:NJL7502L, B.Cu at (73.7, 6.45)
- added Q42: NJL7502L, @Thrive_footprint_kicker:NJL7502L, B.Cu at (-73.7, -6.45)
- added Q43: NJL7502L, @Thrive_footprint_kicker:NJL7502L, B.Cu at (-73.7, 6.45)
- added R100: 1k, Resistor_SMD:R_0805_2012Metric, F.Cu at (148.4, 47.8)
- added R101: 1M, Resistor_SMD:R_0805_2012Metric, F.Cu at (148.4, 50.8)
- added R102: 5.1k, Resistor_SMD:R_0805_2012Metric, F.Cu at (148.4, 53.7)
- added R103: 5.1k, Resistor_SMD:R_0805_2012Metric, F.Cu at (148.4, 56.7)
- added R104: 330, Resistor_SMD:R_0805_2012Metric, F.Cu at (148.4, 59.6)
- added R105: 10k, Resistor_SMD:R_0805_2012Metric, F.Cu at (148.4, 62.6)
- added R83: 75, Resistor_SMD:R_0805_2012Metric, F.Cu at (144.0, 59.6)
- added R87: 10k, Resistor_SMD:R_0805_2012Metric, F.Cu at (144.0, 62.6)
- added R88: 10k, Resistor_SMD:R_0805_2012Metric, F.Cu at (144.0, 65.5)
- added R92: 330, Resistor_SMD:R_0805_2012Metric, F.Cu at (144.0, 68.5)
- added R93: 330, Resistor_SMD:R_0805_2012Metric, F.Cu at (144.0, 71.4)
- added R94: 75, Resistor_SMD:R_0805_2012Metric, F.Cu at (148.4, 39.0)
- added R95: 75, Resistor_SMD:R_0805_2012Metric, F.Cu at (148.4, 41.9)
- added R99: 1k, Resistor_SMD:R_0805_2012Metric, F.Cu at (148.4, 44.9)
- added REF**: MountingHole_3.2mm_M3, MountingHole:MountingHole_3.2mm_M3, F.Cu at (-67.1, -19.7)
- added REF**: MountingHole_3.2mm_M3, MountingHole:MountingHole_3.2mm_M3, F.Cu at (67.1, -19.7)
- added REF**: MountingHole_3.2mm_M3, MountingHole:MountingHole_3.2mm_M3, F.Cu at (-67.1, 19.7)
- added REF**: MountingHole_3.2mm_M3, MountingHole:MountingHole_3.2mm_M3, F.Cu at (67.1, 19.7)
- added REF**: MountingHole_3.2mm_M3, MountingHole:MountingHole_3.2mm_M3, F.Cu at (6.50, -31.9)
- added REF**: MountingHole_3.2mm_M3, MountingHole:MountingHole_3.2mm_M3, F.Cu at (-6.50, -31.9)
- C26: value 100n -> 10μ
- C28: value 10μ -> 100n
- D1, D10, D11, D12, D13, D14, D15, D16, D17, D18, D19, D2, D20, D21, D22, D23, D24, D25, D26, D27, D28, D29, D3, D30, D31, D32, D4, D5, D6, D7, D8, D9, Q1, Q10, Q11, Q12, Q13, Q14, Q15, Q16, Q17, Q18, Q19, Q2, Q20, Q21, Q22, Q23, Q24, Q25, Q26, Q27, Q28, Q29, Q3, Q30, Q31, Q32, Q4, Q5, Q6, Q7, Q8, Q9: moved to B.Cu
- D37: value D40 -> LED; footprint LED_SMD:LED_0603_1608Metric -> LED_THT:LED_D3.0mm; moved to B.Cu
- D38: value D41 -> LED; footprint LED_SMD:LED_0603_1608Metric -> LED_THT:LED_D3.0mm; moved to B.Cu
- R66: value 10k -> 1M
- R69, R70: value 75 -> 10k
- R73: value 10k -> 75
- R74: value 1M -> 75
- R77, R78: value 1k -> 10k
- R82: value 330 -> 75
- moved Q29 350.5 mm to (-44.8, -44.8), turned to 135 degrees
- moved Q28 350.4 mm to (-52.7, -35.2), turned to 146.25 degrees
- moved Q30 349.0 mm to (-35.2, -52.7), turned to 123.75 degrees
- moved Q27 348.7 mm to (-58.5, -24.2), turned to 157.5 degrees
- moved Q26 345.5 mm to (-62.1, -12.4), turned to 168.75 degrees
- moved Q25 340.8 mm to (-63.3, 0.00), turned to 180 degrees
- moved Q24 339.4 mm to (-62.1, 12.4), turned to -168.75 degrees
- moved Q31 333.4 mm to (-24.2, -58.5), turned to 112.5 degrees
- moved Q23 330.2 mm to (-58.5, 24.2), turned to -157.5 degrees
- moved Q32 327.8 mm to (-12.4, -62.1), turned to 101.25 degrees
- moved Q22 319.9 mm to (-52.7, 35.2), turned to -146.25 degrees
- moved Q21 308.5 mm to (-44.8, 44.8), turned to -135 degrees
- moved U17 304.1 mm to (0.00, 0.00), turned to 45 degrees
- moved D28 301.9 mm to (-48.7, -32.6), turned to -33.75 degrees
- moved D29 301.4 mm to (-41.4, -41.4), turned to -45 degrees
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Connections:
- C1 pad 2: +5V_{Line} -> +5VD
- C10 pad 2: +5V_{Line} -> +5VD
- C11 pad 2: +5V_{Line} -> +5VD
- C12 pad 2: +5V_{Line} -> +5VD
- C13 pad 2: +5V_{Line} -> +5VD
- C14 pad 2: +5V_{Line} -> +5VD
- C15 pad 2: +5V_{Line} -> +5VD
- C16 pad 2: +5V_{Line} -> +5VD
- C2 pad 2: +5V_{Line} -> +5VD
- C20 pad 1: +5V_{Line} -> +5VD
- C23 pad 1: +5V_{Line} -> +5VD
- C24 pad 1: Net-(U17-AREF) -> +5VD
- C25 pad 1: +5V_{Line} -> +5VD
- C26 pad 1: +5V_{Line} -> boundary_{backleft}
- C27 pad 1: boundary_{backleft} -> boundary_{frontleft}
- C28 pad 1: boundary_{frontleft} -> Net-(U17-AREF)
- C3 pad 2: +5V_{Line} -> +5VD
- C32 pad 2: +5V_{Line} -> +5VD
- C4 pad 2: +5V_{Line} -> +5VD
- C5 pad 2: +5V_{Line} -> +5VD
- C6 pad 2: +5V_{Line} -> +5VD
- C7 pad 2: +5V_{Line} -> +5VD
- C9 pad 2: +5V_{Line} -> +5VD
- J3 pad 2: +5V_{Line} -> +5VD
- J4 pad A4: VBUS -> Net-(D49-V_{I})
- J4 pad A9: VBUS -> Net-(D49-V_{I})
- J4 pad B4: VBUS -> Net-(D49-V_{I})
- J4 pad B9: VBUS -> Net-(D49-V_{I})
- R65 pad 1: GND -> +5VD
- R65 pad 2: linesig33_{analog} -> RST
- R66 pad 1: GND -> XTAL2
- R66 pad 2: linesig34_{analog} -> XTAL1
- R67 pad 2: linesig35_{analog} -> linesig33_{analog}
- R68 pad 2: linesig36_{analog} -> linesig34_{analog}
- R69 pad 1: Net-(D33-A) -> GND
- R69 pad 2: +5V_{Line} -> linesig35_{analog}
- R70 pad 1: Net-(D34-A) -> GND
- R70 pad 2: +5V_{Line} -> linesig36_{analog}
- R71 pad 1: Net-(D35-A) -> Net-(D33-A)
- R72 pad 1: Net-(D36-A) -> Net-(D34-A)
- R73 pad 1: +5V_{Line} -> Net-(D35-A)
- R73 pad 2: RST -> +5V_{Line}
- R74 pad 1: XTAL2 -> Net-(D36-A)
- R74 pad 2: XTAL1 -> +5V_{Line}
- R77 pad 1: boundary_{backleft_raw} -> GND
- R77 pad 2: boundary_{backleft} -> Net-(Q37-E)
- R78 pad 1: boundary_{frontleft_raw} -> GND
- R78 pad 2: boundary_{frontleft} -> Net-(Q38-E)
- R82 pad 1: VBUS -> Net-(D37-A)
- R82 pad 2: Net-(D39-A) -> +5V_{Line}
- U1 pad 8: +5V_{Line} -> +5VD
- U10 pad 8: +5V_{Line} -> +5VD
- U11 pad 8: +5V_{Line} -> +5VD
- U12 pad 8: +5V_{Line} -> +5VD
- U13 pad 8: +5V_{Line} -> +5VD
- U14 pad 8: +5V_{Line} -> +5VD
- U15 pad 8: +5V_{Line} -> +5VD
- U16 pad 8: +5V_{Line} -> +5VD
- U17 pad 10: +5V_{Line} -> +5VD
- U17 pad 100: +5V_{Line} -> +5VD
- U17 pad 31: +5V_{Line} -> +5VD
- U17 pad 61: +5V_{Line} -> +5VD
- U17 pad 80: +5V_{Line} -> +5VD
- U18 pad 16: +5V_{Line} -> +5VD
- U2 pad 8: +5V_{Line} -> +5VD
- U3 pad 8: +5V_{Line} -> +5VD
- U4 pad 8: +5V_{Line} -> +5VD
- U5 pad 8: +5V_{Line} -> +5VD
- U6 pad 8: +5V_{Line} -> +5VD
- U7 pad 8: +5V_{Line} -> +5VD
- U9 pad 8: +5V_{Line} -> +5VD
Other:
- board size 162.9 x 133.7 mm -> 163.1 x 133.7 mm
- board text added: "裏面部品配置禁止エリア"
- board text removed: "ここら辺にUARTの XHコネクタ配置"

Commit message: Update ラインセンサの部品配置を進めた
Parts:
- removed D47: D40, LED_SMD:LED_0603_1608Metric
- removed D48: D41, LED_SMD:LED_0603_1608Metric
- removed D49: ~, Package_TO_SOT_SMD:TSOT-23
- removed D50: LED_{USB}, LED_SMD:LED_0603_1608Metric
- removed Q42, Q43: NJL7502L, @Thrive_footprint_kicker:NJL7502L
- removed R100, R99: 1k, Resistor_SMD:R_0805_2012Metric
- removed R101: 1M, Resistor_SMD:R_0805_2012Metric
- removed R102, R103: 5.1k, Resistor_SMD:R_0805_2012Metric
- removed R104: 330, Resistor_SMD:R_0805_2012Metric
- removed R105: 10k, Resistor_SMD:R_0805_2012Metric
- removed R94, R95: 75, Resistor_SMD:R_0805_2012Metric
- added D39: LED_Small, LED_THT:LED_D3.0mm, B.Cu at (-69.0, -6.04)
- added D40: LED_Small, LED_THT:LED_D3.0mm, B.Cu at (-69.0, 6.04)
- added D41: LED_Small, LED_SMD:LED_0603_1608Metric, F.Cu at (210.0, 50.5)
- added D44: LED_Small, LED_SMD:LED_0603_1608Metric, F.Cu at (210.0, 55.7)
- added Q39: Q_Photo_NPN_CE, @Thrive_footprint_line:NJL7502L, B.Cu at (-73.7, -6.45)
- added Q40: Q_Photo_NPN_CE, @Thrive_footprint_line:NJL7502L, B.Cu at (-73.7, 6.45)
- added R79: R_Small, Resistor_SMD:R_0805_2012Metric, B.Cu at (-67.3, -10.1)
- added R80: R_Small, Resistor_SMD:R_0805_2012Metric, B.Cu at (-67.3, 10.1)
- added R81: R, Resistor_SMD:R_0805_2012Metric, F.Cu at (190.0, 23.0)
- added R84: R, Resistor_SMD:R_0805_2012Metric, F.Cu at (190.0, 31.8)
- added R85: R_Small, Resistor_SMD:R_0805_2012Metric, F.Cu at (190.0, 34.8)
- added R86: R_Small, Resistor_SMD:R_0805_2012Metric, F.Cu at (190.0, 37.7)
- added R89: R, Resistor_SMD:R_0805_2012Metric, F.Cu at (194.4, 23.0)
- added R90: R, Resistor_SMD:R_0805_2012Metric, F.Cu at (194.4, 25.9)
- added R91: R, Resistor_SMD:R_0805_2012Metric, F.Cu at (194.4, 28.9)
- added SW2: SW_SPDT, @Thrive_footprint_line:SS12D01G4, F.Cu at (74.5, -14.2)
- C1, C10, C11, C12, C13, C14, C15, C16, C2, C28, C3, C31, C33, C4, C5, C6, C7, C8, C9: value 100n -> C_Small
- C17, C19, C29, C30: value 22p -> C
- C18, C23, C24, C25, C32: value 100n -> C
- C20: value 470μ -> C
- C21, C22, C26, C27: value 10μ -> C
- D1, D10, D11, D12, D13, D14, D15, D16, D17, D18, D19, D2, D20, D21, D22, D23, D24, D25, D26, D27, D28, D29, D3, D30, D31, D32, D33, D34, D35, D36, D37, D38, D4, D5, D6, D7, D8, D9: value LED -> LED_Small
- D42: value LED -> LED_Small; footprint LED_THT:LED_D3.0mm -> LED_SMD:LED_0603_1608Metric; moved to F.Cu
- D43: value LED -> ~; footprint LED_THT:LED_D3.0mm -> Package_TO_SOT_SMD:TSOT-23; moved to F.Cu
- J1: value Relay_{Power} -> Conn_01x02_Pin
- J2: value Conn_{Signal} -> Conn_01x02_Pin
- J3: value ICSP_{Arduino} -> Conn_02x03_Odd_Even
- Q1, Q10, Q11, Q12, Q13, Q14, Q15, Q16, Q17, Q18, Q19, Q2, Q20, Q21, Q22, Q23, Q24, Q25, Q26, Q27, Q28, Q29, Q3, Q30, Q31, Q32, Q33, Q34, Q35, Q36, Q37, Q38, Q4, Q5, Q6, Q7, Q8, Q9: value NJL7502L -> Q_Photo_NPN_CE; footprint @Thrive_footprint_kicker:NJL7502L -> @Thrive_footprint_line:NJL7502L
- R1, R11, R12, R13, R14, R15, R2, R21, R22, R23, R24, R25, R3, R31, R32, R4, R41, R42, R43, R44, R45, R5, R51, R52, R53, R54, R55, R61, R62, R65, R67, R68, R69, R70, R77, R78: value 10k -> R_Small; moved to B.Cu
- R10, R16, R17, R18, R19, R20, R26, R27, R28, R29, R30, R38, R40, R46, R47, R48, R49, R50, R56, R57, R58, R59, R6, R60, R63, R64, R7, R71, R72, R8, R9: value 75 -> R_Small; moved to B.Cu
- R33, R34, R35: value 10k -> R_Small
- R36, R37, R39, R73, R74: value 75 -> R_Small
- R66: value 1M -> R_Small; moved to B.Cu
- R75, R76: value 1k -> R_Small
- R82, R83: value 75 -> R
- R87, R88: value 10k -> R
- R92: value 330 -> R_Small
- R93: value 330 -> R
- SW1: value RESET -> SW_Push
- U1, U10, U11, U12, U13, U14, U15, U16, U2, U3, U4, U5, U6, U7, U8, U9: value LM339DR -> LM393DR; footprint Package_SO:SOIC-14_3.9x8.7mm_P1.27mm -> Package_SO:SOIC-8_3.9x4.9mm_P1.27mm
- U18: moved to B.Cu
- Y1: value 16MHz -> Crystal
- Y2: value 12MHz -> Crystal
- moved D42 285.2 mm to (210.0, 53.1), turned to 0 degrees
- moved R40 212.2 mm to (-73.2, -10.9), turned to -8.5 degrees
- moved R67 208.9 mm to (-51.6, -27.6), turned to 151.875 degrees
- moved R68 208.6 mm to (-45.2, -37.1), turned to 140.625 degrees
- moved C14 208.1 mm to (-48.9, -26.2), turned to -118.125 degrees
- moved R66 207.9 mm to (-56.0, -17.0), turned to 163.125 degrees
- moved R69 207.0 mm to (-37.1, -45.2), turned to 129.375 degrees
- moved R65 205.7 mm to (-58.2, -5.73), turned to 174.375 degrees
- moved R70 204.1 mm to (-27.6, -51.6), turned to 118.125 degrees
- moved R64 202.2 mm to (-58.2, 5.73), turned to -174.375 degrees
- moved C13 201.0 mm to (-55.2, -5.44), turned to -95.625 degrees
- moved R71 200.0 mm to (-17.0, -56.0), turned to 106.875 degrees
- moved C15 199.7 mm to (-35.2, -42.9), turned to -140.625 degrees
- moved R63 197.5 mm to (-56.0, 17.0), turned to -163.125 degrees
- moved R27 196.1 mm to (-55.1, -29.5), turned to -28.125 degrees
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Connections:
- C8 pad 2: +5V_{Line} -> +5VD
- D43 pad 2: Net-(D43-A) -> VBUS
- J4 pad A4: Net-(D49-V_{I}) -> Net-(D43-V_{I})
- J4 pad A9: Net-(D49-V_{I}) -> Net-(D43-V_{I})
- J4 pad B4: Net-(D49-V_{I}) -> Net-(D43-V_{I})
- J4 pad B9: Net-(D49-V_{I}) -> Net-(D43-V_{I})
- Q37 pad 2: Net-(Q37-E) -> linesig1^{side}_{raw}
- Q38 pad 2: Net-(Q38-E) -> linesig1^{side}_{raw}
- R1 pad 1: GND -> linesig1_{raw}
- R1 pad 2: linesig1_{raw} -> GND
- R10 pad 1: Net-(D5-A) -> linesig10_{raw}
- R10 pad 2: +5V_{Line} -> GND
- R11 pad 1: GND -> linesig11_{raw}
- R11 pad 2: linesig6_{raw} -> GND
- R12 pad 1: GND -> linesig12_{raw}
- R12 pad 2: linesig7_{raw} -> GND
- R13 pad 1: GND -> linesig13_{raw}
- R13 pad 2: linesig8_{raw} -> GND
- R14 pad 1: GND -> linesig14_{raw}
- R14 pad 2: linesig9_{raw} -> GND
- R15 pad 1: GND -> linesig15_{raw}
- R15 pad 2: linesig10_{raw} -> GND
- R16 pad 1: Net-(D6-A) -> linesig16_{raw}
- R16 pad 2: +5V_{Line} -> GND
- R17 pad 1: Net-(D7-A) -> linesig17_{raw}
- R17 pad 2: +5V_{Line} -> GND
- R18 pad 1: Net-(D8-A) -> linesig18_{raw}
- R18 pad 2: +5V_{Line} -> GND
- R19 pad 1: Net-(D9-A) -> linesig19_{raw}
- R19 pad 2: +5V_{Line} -> GND
- R2 pad 1: GND -> linesig2_{raw}
- R2 pad 2: linesig2_{raw} -> GND
- R20 pad 1: Net-(D10-A) -> linesig20_{raw}
- R20 pad 2: +5V_{Line} -> GND
- R21 pad 1: GND -> linesig21_{raw}
- R21 pad 2: linesig11_{raw} -> GND
- R22 pad 1: GND -> linesig22_{raw}
- R22 pad 2: linesig12_{raw} -> GND
- R23 pad 1: GND -> linesig23_{raw}
- R23 pad 2: linesig13_{raw} -> GND
- R24 pad 1: GND -> linesig24_{raw}
- R24 pad 2: linesig14_{raw} -> GND
- R25 pad 1: GND -> linesig25_{raw}
- R25 pad 2: linesig15_{raw} -> GND
- R26 pad 1: Net-(D11-A) -> linesig26_{raw}
- R26 pad 2: +5V_{Line} -> GND
- R27 pad 1: Net-(D12-A) -> linesig27_{raw}
- R27 pad 2: +5V_{Line} -> GND
- R28 pad 1: Net-(D13-A) -> linesig28_{raw}
- R28 pad 2: +5V_{Line} -> GND
- R29 pad 1: Net-(D14-A) -> linesig29_{raw}
- R29 pad 2: +5V_{Line} -> GND
- R3 pad 1: GND -> linesig3_{raw}
- R3 pad 2: linesig3_{raw} -> GND
- R30 pad 1: Net-(D15-A) -> linesig30_{raw}
- R30 pad 2: +5V_{Line} -> GND
- R31 pad 1: GND -> linesig31_{raw}
- R31 pad 2: linesig16_{raw} -> GND
- R32 pad 1: GND -> linesig32_{raw}
- R32 pad 2: linesig17_{raw} -> GND
- R33 pad 1: GND -> linesig33_{analog}
- R33 pad 2: linesig18_{raw} -> GND
- R34 pad 1: GND -> linesig34_{analog}
- R34 pad 2: linesig19_{raw} -> GND
- R35 pad 1: GND -> linesig35_{analog}
- R35 pad 2: linesig20_{raw} -> GND
- R36 pad 1: Net-(D16-A) -> linesig36_{analog}
- R36 pad 2: +5V_{Line} -> GND
- R37 pad 1: Net-(D17-A) -> linesig1^{side}_{raw}
- R37 pad 2: +5V_{Line} -> GND
- R38 pad 1: Net-(D18-A) -> linesig1^{side}_{raw}
- R38 pad 2: +5V_{Line} -> GND
- R39 pad 1: Net-(D19-A) -> linesig2^{side}_{raw}
- R39 pad 2: +5V_{Line} -> GND
- R4 pad 1: GND -> linesig4_{raw}
- R4 pad 2: linesig4_{raw} -> GND
- R40 pad 1: Net-(D20-A) -> linesig2^{side}_{raw}
- R40 pad 2: +5V_{Line} -> GND
- R41 pad 1: GND -> Net-(D1-A)
- R41 pad 2: linesig21_{raw} -> +5V_{Line}
- R42 pad 1: GND -> Net-(D2-A)
- R42 pad 2: linesig22_{raw} -> +5V_{Line}
- R43 pad 1: GND -> Net-(D3-A)
- R43 pad 2: linesig23_{raw} -> +5V_{Line}
- R44 pad 1: GND -> Net-(D4-A)
- R44 pad 2: linesig24_{raw} -> +5V_{Line}
- R45 pad 1: GND -> Net-(D5-A)
- R45 pad 2: linesig25_{raw} -> +5V_{Line}
- R46 pad 1: Net-(D21-A) -> Net-(D6-A)
- R47 pad 1: Net-(D22-A) -> Net-(D7-A)
- R48 pad 1: Net-(D23-A) -> Net-(D8-A)
- R49 pad 1: Net-(D24-A) -> Net-(D9-A)
- R5 pad 1: GND -> linesig5_{raw}
- R5 pad 2: linesig5_{raw} -> GND
- R50 pad 1: Net-(D25-A) -> Net-(D10-A)
- R51 pad 1: GND -> Net-(D11-A)
- R51 pad 2: linesig26_{raw} -> +5V_{Line}
- R52 pad 1: GND -> Net-(D12-A)
- R52 pad 2: linesig27_{raw} -> +5V_{Line}
- R53 pad 1: GND -> Net-(D13-A)
- R53 pad 2: linesig28_{raw} -> +5V_{Line}
- R54 pad 1: GND -> Net-(D14-A)
- R54 pad 2: linesig29_{raw} -> +5V_{Line}
- R55 pad 1: GND -> Net-(D15-A)
- R55 pad 2: linesig30_{raw} -> +5V_{Line}
- R56 pad 1: Net-(D26-A) -> Net-(D16-A)
- R57 pad 1: Net-(D27-A) -> Net-(D17-A)
- R58 pad 1: Net-(D28-A) -> Net-(D18-A)
- R59 pad 1: Net-(D29-A) -> Net-(D19-A)
- R6 pad 1: Net-(D1-A) -> linesig6_{raw}
- R6 pad 2: +5V_{Line} -> GND
- R60 pad 1: Net-(D30-A) -> Net-(D20-A)
- R61 pad 1: GND -> Net-(D21-A)
- R61 pad 2: linesig31_{raw} -> +5V_{Line}
- R62 pad 1: GND -> Net-(D22-A)
- R62 pad 2: linesig32_{raw} -> +5V_{Line}
- R63 pad 1: Net-(D31-A) -> Net-(D23-A)
- R64 pad 1: Net-(D32-A) -> Net-(D24-A)
- R65 pad 1: +5VD -> Net-(D25-A)
- R65 pad 2: RST -> +5V_{Line}
- R66 pad 1: XTAL2 -> Net-(D26-A)
- R66 pad 2: XTAL1 -> +5V_{Line}
- R67 pad 1: GND -> Net-(D27-A)
- R67 pad 2: linesig33_{analog} -> +5V_{Line}
- R68 pad 1: GND -> Net-(D28-A)
- R68 pad 2: linesig34_{analog} -> +5V_{Line}
- R69 pad 1: GND -> Net-(D29-A)
- R69 pad 2: linesig35_{analog} -> +5V_{Line}
- R7 pad 1: Net-(D2-A) -> linesig7_{raw}
- R7 pad 2: +5V_{Line} -> GND
- R70 pad 1: GND -> Net-(D30-A)
- R70 pad 2: linesig36_{analog} -> +5V_{Line}
- R71 pad 1: Net-(D33-A) -> Net-(D31-A)
- R72 pad 1: Net-(D34-A) -> Net-(D32-A)
- R73 pad 1: Net-(D35-A) -> Net-(D33-A)
- R74 pad 1: Net-(D36-A) -> Net-(D34-A)
- R75 pad 1: boundary_{frontright_raw} -> Net-(D35-A)
- R75 pad 2: boundary_{frontright} -> +5V_{Line}
- R76 pad 1: boundary_{backright_raw} -> Net-(D36-A)
- R76 pad 2: boundary_{backright} -> +5V_{Line}
- R77 pad 1: GND -> Net-(D37-A)
- R77 pad 2: Net-(Q37-E) -> +5V_{Line}
- R78 pad 1: GND -> Net-(D38-A)
- R78 pad 2: Net-(Q38-E) -> +5V_{Line}
- R8 pad 1: Net-(D3-A) -> linesig8_{raw}
- R8 pad 2: +5V_{Line} -> GND
- R82 pad 1: Net-(D37-A) -> XTAL2
- R82 pad 2: +5V_{Line} -> XTAL1
- R83 pad 1: Net-(D38-A) -> boundary_{frontright_raw}
- R83 pad 2: +5V_{Line} -> boundary_{frontright}
- R87 pad 1: GND -> boundary_{backleft_raw}
- R87 pad 2: Net-(Q42-E) -> boundary_{backleft}
- R88 pad 1: GND -> boundary_{frontleft_raw}
- R88 pad 2: Net-(Q43-E) -> boundary_{frontleft}
- R9 pad 1: Net-(D4-A) -> linesig9_{raw}
- R9 pad 2: +5V_{Line} -> GND
- R92 pad 1: LED1 -> VBUS
- R93 pad 1: LED2 -> Net-(U18-~{DTR})
- R93 pad 2: Net-(D48-A) -> GND
- U1 pad 1: linesig1_{digital} -> linesig2_{digital}
- U1 pad 3: linesig1_{raw} -> linesig2_{raw}
- U1 pad 5: linesig2_{raw} -> linesig1_{raw}
- U1 pad 7: linesig2_{digital} -> linesig1_{digital}
- U10 pad 1: linesig19_{digital} -> linesig20_{digital}
- U10 pad 3: linesig19_{raw} -> linesig20_{raw}
- U10 pad 5: linesig20_{raw} -> linesig19_{raw}
- U10 pad 7: linesig20_{digital} -> linesig19_{digital}
- U11 pad 1: linesig21_{digital} -> linesig22_{digital}
- U11 pad 3: linesig21_{raw} -> linesig22_{raw}
- U11 pad 5: linesig22_{raw} -> linesig21_{raw}
- U11 pad 7: linesig22_{digital} -> linesig21_{digital}
- U12 pad 1: linesig23_{digital} -> linesig24_{digital}
- U12 pad 3: linesig23_{raw} -> linesig24_{raw}
- U12 pad 5: linesig24_{raw} -> linesig23_{raw}
- U12 pad 7: linesig24_{digital} -> linesig23_{digital}
- U13 pad 1: linesig25_{digital} -> linesig26_{digital}
- U13 pad 3: linesig25_{raw} -> linesig26_{raw}
- U13 pad 5: linesig26_{raw} -> linesig25_{raw}
- U13 pad 7: linesig26_{digital} -> linesig25_{digital}
- U14 pad 1: linesig27_{digital} -> linesig28_{digital}
- U14 pad 3: linesig27_{raw} -> linesig28_{raw}
- U14 pad 5: linesig28_{raw} -> linesig27_{raw}
- U14 pad 7: linesig28_{digital} -> linesig27_{digital}
- U15 pad 1: linesig29_{digital} -> linesig30_{digital}
- U15 pad 3: linesig29_{raw} -> linesig30_{raw}
- U15 pad 5: linesig30_{raw} -> linesig29_{raw}
- U15 pad 7: linesig30_{digital} -> linesig29_{digital}
- U16 pad 1: linesig31_{digital} -> linesig32_{digital}
- U16 pad 3: linesig31_{raw} -> linesig32_{raw}
- U16 pad 5: linesig32_{raw} -> linesig31_{raw}
- U16 pad 7: linesig32_{digital} -> linesig31_{digital}
- U2 pad 1: linesig3_{digital} -> linesig4_{digital}
- U2 pad 3: linesig3_{raw} -> linesig4_{raw}
- U2 pad 5: linesig4_{raw} -> linesig3_{raw}
- U2 pad 7: linesig4_{digital} -> linesig3_{digital}
- U3 pad 1: linesig5_{digital} -> linesig6_{digital}
- U3 pad 3: linesig5_{raw} -> linesig6_{raw}
- U3 pad 5: linesig6_{raw} -> linesig5_{raw}
- U3 pad 7: linesig6_{digital} -> linesig5_{digital}
- U4 pad 1: linesig7_{digital} -> linesig8_{digital}
- U4 pad 3: linesig7_{raw} -> linesig8_{raw}
- U4 pad 5: linesig8_{raw} -> linesig7_{raw}
- U4 pad 7: linesig8_{digital} -> linesig7_{digital}
- U5 pad 1: linesig9_{digital} -> linesig10_{digital}
- U5 pad 3: linesig9_{raw} -> linesig10_{raw}
- U5 pad 5: linesig10_{raw} -> linesig9_{raw}
- U5 pad 7: linesig10_{digital} -> linesig9_{digital}
- U6 pad 1: linesig11_{digital} -> linesig12_{digital}
- U6 pad 3: linesig11_{raw} -> linesig12_{raw}
- U6 pad 5: linesig12_{raw} -> linesig11_{raw}
- U6 pad 7: linesig12_{digital} -> linesig11_{digital}
- U7 pad 1: linesig13_{digital} -> linesig14_{digital}
- U7 pad 3: linesig13_{raw} -> linesig14_{raw}
- U7 pad 5: linesig14_{raw} -> linesig13_{raw}
- U7 pad 7: linesig14_{digital} -> linesig13_{digital}
- U8 pad 1: linesig15_{digital} -> linesig16_{digital}
- U8 pad 3: linesig15_{raw} -> linesig16_{raw}
- U8 pad 5: linesig16_{raw} -> linesig15_{raw}
- U8 pad 7: linesig16_{digital} -> linesig15_{digital}
- U8 pad 8: +5V_{Line} -> +5VD
- U9 pad 1: linesig17_{digital} -> linesig18_{digital}
- U9 pad 3: linesig17_{raw} -> linesig18_{raw}
- U9 pad 5: linesig18_{raw} -> linesig17_{raw}
- U9 pad 7: linesig18_{digital} -> linesig17_{digital}
Routing:
- net +5V_{Line}: track 0.00 -> 471.2 mm
- net linesig2^{side}_{raw}: track 0.00 -> 17.7 mm
- net linesig1^{side}_{raw}: track 0.00 -> 17.7 mm
- net linesig32_{raw}: track 0.00 -> 6.39 mm
- net linesig31_{raw}: track 0.00 -> 6.39 mm
- net linesig1_{raw}: track 0.00 -> 6.39 mm
- net linesig30_{raw}: track 0.00 -> 6.39 mm
- net linesig2_{raw}: track 0.00 -> 6.39 mm
- net linesig29_{raw}: track 0.00 -> 6.39 mm
- net linesig3_{raw}: track 0.00 -> 6.39 mm
- net linesig28_{raw}: track 0.00 -> 6.39 mm
- net linesig4_{raw}: track 0.00 -> 6.39 mm
- net linesig27_{raw}: track 0.00 -> 6.39 mm
- net linesig5_{raw}: track 0.00 -> 6.39 mm
- net linesig26_{raw}: track 0.00 -> 6.39 mm
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- added copper zone on B.Cu, net GND
- added copper zone on F.Cu, net GND

Commit message: Update ラインセンサ基板の配線を進めた
Parts:
- removed R37, R39: R_Small, Resistor_SMD:R_0805_2012Metric
- added C34: 100n, Capacitor_SMD:C_0805_2012Metric, F.Cu at (9.78, 1.16)
- added C35: 100n, Capacitor_SMD:C_0805_2012Metric, F.Cu at (5.50, 10.1)
- added C36: 100n, Capacitor_SMD:C_0805_2012Metric, F.Cu at (-4.00, 10.1)
- added C37: 100n, Capacitor_SMD:C_0805_2012Metric, F.Cu at (-10.4, -0.84)
- added C38: 100n, Capacitor_SMD:C_0805_2012Metric, F.Cu at (3.00, -10.2)
- R1, R10, R11, R12, R13, R14, R15, R16, R17, R18, R19, R2, R20, R21, R22, R23, R24, R25, R26, R27, R28, R29, R3, R30, R31, R32, R4, R41, R42, R43, R44, R45, R46, R47, R48, R49, R5, R50, R51, R52, R53, R54, R55, R56, R57, R58, R59, R6, R60, R61, R62, R63, R64, R65, R66, R67, R68, R69, R7, R70, R71, R72, R8, R9: moved to F.Cu
- moved C29 233.7 mm to (135.6, 243.3), turned to -45 degrees
- moved C30 233.6 mm to (133.5, 245.4), turned to -45 degrees
- moved C31 233.5 mm to (131.4, 247.6), turned to -45 degrees
- moved C32 233.4 mm to (129.3, 249.7), turned to -45 degrees
- moved C33 233.4 mm to (127.1, 251.8), turned to -45 degrees
- moved C23 230.3 mm to (132.5, 240.2), turned to -45 degrees
- moved C24 230.2 mm to (130.4, 242.3), turned to -45 degrees
- moved C25 230.1 mm to (128.2, 244.4), turned to -45 degrees
- moved C26 230.0 mm to (126.1, 246.5), turned to -45 degrees
- moved C27 230.0 mm to (124.0, 248.7), turned to -45 degrees
- moved C28 230.0 mm to (121.9, 250.8), turned to -45 degrees
- moved Y1 228.4 mm to (96.5, 243.5), turned to -45 degrees
- moved R89 226.9 mm to (122.1, 238.0), turned to -45 degrees
- moved C17 226.9 mm to (129.4, 237.0), turned to -45 degrees
- moved C18 226.8 mm to (127.2, 239.1), turned to -45 degrees
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Connections:
- U17 pad 14: unconnected-(U17-PH2-Pad14) -> linesig10_{digital}
- U17 pad 15: linesig1_{digital} -> linesig9_{digital}
- U17 pad 16: linesig2_{digital} -> linesig8_{digital}
- U17 pad 17: linesig3_{digital} -> linesig7_{digital}
- U17 pad 18: linesig4_{digital} -> linesig6_{digital}
- U17 pad 19: unconnected-(U17-PB0-Pad19) -> linesig5_{digital}
- U17 pad 23: linesig5_{digital} -> linesig4_{digital}
- U17 pad 24: linesig6_{digital} -> linesig3_{digital}
- U17 pad 25: linesig7_{digital} -> linesig2_{digital}
- U17 pad 26: linesig8_{digital} -> linesig1_{digital}
- U17 pad 27: unconnected-(U17-PH7-Pad27) -> linesig32_{digital}
- U17 pad 28: unconnected-(U17-PG3-Pad28) -> linesig31_{digital}
- U17 pad 35: unconnected-(U17-PL0-Pad35) -> linesig30_{digital}
- U17 pad 36: unconnected-(U17-PL1-Pad36) -> linesig29_{digital}
- U17 pad 37: unconnected-(U17-PL2-Pad37) -> linesig28_{digital}
- U17 pad 38: unconnected-(U17-PL3-Pad38) -> linesig27_{digital}
- U17 pad 43: linesig14_{digital} -> unconnected-(U17-PD0-Pad43)
- U17 pad 44: linesig13_{digital} -> unconnected-(U17-PD1-Pad44)
- U17 pad 45: linesig12_{digital} -> unconnected-(U17-PD2-Pad45)
- U17 pad 46: linesig11_{digital} -> unconnected-(U17-PD3-Pad46)
- U17 pad 50: linesig31_{digital} -> unconnected-(U17-PD7-Pad50)
- U17 pad 51: LED2 -> linesig26_{digital}
- U17 pad 52: LED1 -> linesig25_{digital}
- U17 pad 53: linesig30_{digital} -> linesig24_{digital}
- U17 pad 54: linesig29_{digital} -> linesig23_{digital}
- U17 pad 55: linesig28_{digital} -> linesig22_{digital}
- U17 pad 56: linesig27_{digital} -> linesig21_{digital}
- U17 pad 57: linesig26_{digital} -> linesig20_{digital}
- U17 pad 58: linesig25_{digital} -> linesig19_{digital}
- U17 pad 59: linesig24_{digital} -> unconnected-(U17-PC6-Pad59)
- U17 pad 60: linesig23_{digital} -> unconnected-(U17-PC7-Pad60)
- U17 pad 63: linesig10_{digital} -> unconnected-(U17-PJ0-Pad63)
- U17 pad 64: linesig9_{digital} -> unconnected-(U17-PJ1-Pad64)
- U17 pad 66: unconnected-(U17-PJ3-Pad66) -> linesig18_{digital}
- U17 pad 67: unconnected-(U17-PJ4-Pad67) -> linesig17_{digital}
- U17 pad 70: linesig32_{digital} -> unconnected-(U17-PG2-Pad70)
- U17 pad 71: linesig22_{digital} -> unconnected-(U17-PA7-Pad71)
- U17 pad 72: linesig21_{digital} -> unconnected-(U17-PA6-Pad72)
- U17 pad 73: linesig20_{digital} -> unconnected-(U17-PA5-Pad73)
- U17 pad 74: linesig19_{digital} -> linesig16_{digital}
- U17 pad 75: linesig18_{digital} -> linesig15_{digital}
- U17 pad 76: linesig17_{digital} -> linesig14_{digital}
- U17 pad 77: linesig16_{digital} -> linesig13_{digital}
- U17 pad 78: linesig15_{digital} -> unconnected-(U17-PA0-Pad78)
- U17 pad 90: unconnected-(U17-PF7-Pad90) -> linesig12_{digital}
- U17 pad 91: unconnected-(U17-PF6-Pad91) -> linesig11_{digital}
- U17 pad 94: linesig36_{analog} -> unconnected-(U17-PF3-Pad94)
- U17 pad 95: linesig35_{analog} -> unconnected-(U17-PF2-Pad95)
- U17 pad 96: linesig34_{analog} -> unconnected-(U17-PF1-Pad96)
- U17 pad 97: linesig33_{analog} -> unconnected-(U17-PF0-Pad97)
Routing:
- net +5VD: track 0.00 -> 520.0 mm, vias 0 -> 17
- net +5V_{Line}: track 471.2 -> 607.7 mm, vias 0 -> 16
- net boundary_{backleft}: track 0.00 -> 77.0 mm
- net boundary_{frontleft}: track 0.00 -> 77.0 mm
- net boundary_{backright}: track 0.00 -> 77.0 mm
- net boundary_{frontright}: track 0.00 -> 77.0 mm
- net linesig9_{digital}: track 0.00 -> 63.3 mm
- net linesig27_{digital}: track 0.00 -> 61.4 mm
- net linesig10_{digital}: track 0.00 -> 60.8 mm
- net linesig19_{digital}: track 0.00 -> 59.0 mm
- net linesig7_{digital}: track 0.00 -> 58.8 mm
- net linesig25_{digital}: track 0.00 -> 58.6 mm
- net RX_{teensy}-TX_{Arduino}-5V: track 0.00 -> 58.4 mm, vias 0 -> 1
- net linesig11_{digital}: track 0.00 -> 57.3 mm
- net linesig28_{digital}: track 0.00 -> 57.1 mm
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Other:
- board size 163.1 x 133.7 mm -> 137.8 x 137.8 mm
