File: circuit/line-001-20260628/line-001-20260628.kicad_pcb (KiCad board)
At the start: 2 copper layers, 137.8 x 137.8 mm, 245 parts, among them J1 Conn_01x02_Pin, J2 Conn_01x02_Pin, J3 Conn_02x03_Odd_Even, J4 USB_C_Receptacle_USB2.0_16P, Q1 Q_Photo_NPN_CE, Q10 Q_Photo_NPN_CE, Q11 Q_Photo_NPN_CE, Q12 Q_Photo_NPN_CE, Q13 Q_Photo_NPN_CE, Q14 Q_Photo_NPN_CE, Q15 Q_Photo_NPN_CE, Q16 Q_Photo_NPN_CE, Q17 Q_Photo_NPN_CE, Q18 Q_Photo_NPN_CE, Q19 Q_Photo_NPN_CE, Q2 Q_Photo_NPN_CE, Q20 Q_Photo_NPN_CE, Q21 Q_Photo_NPN_CE, Q22 Q_Photo_NPN_CE, Q23 Q_Photo_NPN_CE, Q24 Q_Photo_NPN_CE, Q25 Q_Photo_NPN_CE, Q26 Q_Photo_NPN_CE, Q27 Q_Photo_NPN_CE, Q28 Q_Photo_NPN_CE, Q29 Q_Photo_NPN_CE, Q3 Q_Photo_NPN_CE, Q30 Q_Photo_NPN_CE, Q31 Q_Photo_NPN_CE, Q32 Q_Photo_NPN_CE, Q33 Q_Photo_NPN_CE, Q34 Q_Photo_NPN_CE, Q35 Q_Photo_NPN_CE, Q36 Q_Photo_NPN_CE, Q37 Q_Photo_NPN_CE, Q38 Q_Photo_NPN_CE, Q39 Q_Photo_NPN_CE, Q4 Q_Photo_NPN_CE, Q40 Q_Photo_NPN_CE, Q5 Q_Photo_NPN_CE, Q6 Q_Photo_NPN_CE, Q7 Q_Photo_NPN_CE, Q8 Q_Photo_NPN_CE, Q9 Q_Photo_NPN_CE, SW1 SW_Push, SW2 SW_SPDT, U1 LM393DR, U10 LM393DR, U11 LM393DR, U12 LM393DR, U13 LM393DR, U14 LM393DR, U15 LM393DR, U16 LM393DR, U17 ATmega2560-16A, U18 CH340G, U2 LM393DR, U3 LM393DR, U4 LM393DR, U5 LM393DR, U6 LM393DR, U7 LM393DR, U8 LM393DR, U9 LM393DR, Y1 Crystal, Y2 Crystal

Commit message: Update ラインセンサ基板を進めた、GND孤立がひどい
Parts:
- removed C23, C24, C25: C, Capacitor_SMD:C_0805_2012Metric
- removed D33, D34, D35, D36: LED_Small, LED_THT:LED_D3.0mm
- removed Q33, Q34, Q35, Q36: Q_Photo_NPN_CE, @Thrive_footprint_line:NJL7502L
- removed R33, R34, R35, R36, R73, R74, R75, R76: R_Small, Resistor_SMD:R_0805_2012Metric
- C1, C10, C11, C12, C13, C14, C15, C16, C2, C28, C3, C33, C4, C5, C6, C7, C8, C9: value C_Small -> 100n
- C17, C19, C29, C30: value C -> 22p; footprint Capacitor_SMD:C_0805_2012Metric -> Capacitor_SMD:C_0603_1608Metric
- C18, C32: value C -> 100n
- C20: value C -> 100μ; footprint Capacitor_SMD:C_0805_2012Metric -> Capacitor_SMD:C_1206_3216Metric
- D41: value LED_Small -> LED1
- D42: value LED_Small -> LED2
- D44: value LED_Small -> USB
- R1, R10, R11, R12, R13, R14, R15, R16, R17, R18, R19, R2, R20, R21, R22, R23, R24, R25, R26, R27, R28, R29, R3, R30, R31, R32, R4, R5, R6, R7, R8, R9: value R_Small -> 10k
- R38, R40: value R_Small -> 10k; moved to F.Cu
- R41, R42, R43, R44, R45, R46, R47, R48, R49, R50, R51, R52, R53, R54, R55, R56, R57, R58, R59, R60, R61, R62, R63, R64, R65, R66, R67, R68, R69, R70, R71, R72: value R_Small -> 75
- R77, R78, R79, R80: value R_Small -> 75; moved to F.Cu
- R81: value R -> 10k
- R82, R89: value R -> 1M
- R85, R86, R92: value R_Small -> 330
- R90, R91: value R -> 5.1k
- R93: value R -> 4.7k
- Y1: value Crystal -> 16MHz; footprint Crystal:Crystal_HC49-4H_Vertical -> Crystal:Crystal_SMD_SeikoEpson_FA238-4Pin_3.2x2.5mm; moved to B.Cu
- Y2: value Crystal -> 12MHz; footprint Crystal:Crystal_HC49-4H_Vertical -> Crystal:Crystal_SMD_SeikoEpson_FA238V-4Pin_3.2x2.5mm; moved to B.Cu
- moved C17 283.1 mm to (-3.48, -13.0), turned to 135 degrees
- moved C19 282.3 mm to (-9.84, -6.66)
- moved R82 279.0 mm to (-8.60, -13.2), turned to 135 degrees
- moved Y1 273.5 mm to (-6.66, -9.84), turned to -135 degrees
- moved C27 272.5 mm to (14.1, -0.71), turned to -135 degrees
- moved C22 271.0 mm to (17.0, -3.54), turned to -135 degrees
- moved C28 269.4 mm to (9.72, 5.83)
- moved C26 267.2 mm to (17.3, 2.48), turned to -135 degrees
- moved R84 263.4 mm to (15.6, -4.95), turned to 45 degrees
- moved R88 262.8 mm to (12.7, -2.12), turned to 45 degrees
- moved C33 259.9 mm to (78.8, -3.50), turned to 0 degrees
- moved R87 257.6 mm to (15.9, 1.06), turned to 45 degrees
- moved C32 255.8 mm to (73.5, 0.00), turned to 90 degrees
- moved C18 254.1 mm to (77.8, -10.1), turned to -82.6 degrees
- moved C31 253.8 mm to (84.0, -1.75), turned to -90 degrees
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Connections:
- Y1 pad 2: XTAL1 -> (no net)
- Y2 pad 2: Net-(U18-XI) -> (no net)
Routing:
- net TX_{Arduino}: track 0.00 -> 91.8 mm, vias 0 -> 3
- net RX_{Arduino}: track 0.00 -> 89.8 mm, vias 0 -> 3
- net boundary_{frontleft}: track 77.0 -> 162.0 mm, vias 0 -> 2
- net RST: track 24.5 -> 105.7 mm, vias 1 -> 3
- net boundary_{backleft}: track 77.0 -> 148.1 mm, vias 0 -> 2
- net boundary_{backright}: track 77.0 -> 128.4 mm
- net boundary_{frontright}: track 77.0 -> 124.8 mm, vias 0 -> 2
- net +5VD: track 520.0 -> 559.8 mm, vias 17 -> 21
- net Net-(U18-XO): track 0.00 -> 28.1 mm, vias 0 -> 1
- net Net-(U18-XI): track 0.00 -> 21.5 mm, vias 0 -> 1
- net +5V_{Line}: track 607.7 -> 627.1 mm, vias 16 -> 18
- net XTAL1: track 0.00 -> 17.4 mm, vias 0 -> 3
- net XTAL2: track 0.00 -> 16.3 mm, vias 0 -> 3
- net VBUS: track 13.1 -> 27.7 mm
- net boundary_{frontright_raw}: track 0.00 -> 12.0 mm
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Other:
- board size 137.8 x 137.8 mm -> 163.1 x 133.7 mm

Commit message: Update ラインセンサ基板のPCBを進めた
Routing:
- net boundary_{backright}: track 128.4 -> 159.5 mm, vias 0 -> 8
- net boundary_{backleft}: track 148.1 -> 162.3 mm, vias 2 -> 10
- net boundary_{frontleft}: track 162.0 -> 175.8 mm, vias 2 -> 10
- net boundary_{frontright}: track 124.8 -> 134.5 mm, vias 2 -> 10
- net XTAL2: track 16.3 -> 18.1 mm
- net linesig27_{digital}: track 61.4 -> 60.9 mm
- net linesig32_{digital}: track 52.8 -> 53.2 mm, vias 0 -> 2
- net linesig31_{digital}: track 55.9 -> 56.2 mm, vias 0 -> 2
- net GND: vias 13 -> 93

Commit message: Update ラインセンサ基板のシルクスクリーンを整えてLEDを取り付けた
Parts:
- C31: value C_Small -> 100n
- D41, D42: moved to B.Cu
- J3: value Conn_02x03_Odd_Even -> ICSP
- Y1: moved to F.Cu
- moved D41 153.6 mm to (-1.25, 14.0), turned to -90 degrees
- moved D42 151.7 mm to (1.25, 14.0), turned to -90 degrees
- moved R85 149.5 mm to (-1.25, 14.0), turned to -90 degrees
- moved R86 147.7 mm to (1.25, 14.0), turned to -90 degrees
- moved C19 13.6 mm to (-9.25, -20.2), turned to 90 degrees
- moved Y1 10.4 mm to (-6.25, -20.2), turned to 180 degrees
- moved R82 10.3 mm to (-6.25, -23.2), turned to 180 degrees
- moved C17 7.23 mm to (-3.25, -20.2), turned to -90 degrees
Connections:
- U17 pad 68: unconnected-(U17-PJ5-Pad68) -> linesig16_{digital}
- U17 pad 69: unconnected-(U17-PJ6-Pad69) -> linesig15_{digital}
- U17 pad 74: linesig16_{digital} -> LED1
- U17 pad 75: linesig15_{digital} -> LED2
Routing:
- net XTAL1: track 17.4 -> 23.8 mm, vias 3 -> 2
- net XTAL2: track 18.1 -> 24.1 mm, vias 3 -> 2
- net LED2: track 0.00 -> 4.43 mm
- net LED1: track 0.00 -> 4.35 mm
- net linesig15_{digital}: track 56.3 -> 60.3 mm
- net linesig16_{digital}: track 54.5 -> 58.1 mm
- net Net-(D42-A): track 0.00 -> 2.30 mm, vias 0 -> 1
- net Net-(D41-A): track 0.00 -> 2.30 mm, vias 0 -> 1
- net linesig32_{digital}: track 53.2 -> 52.8 mm, vias 2 -> 0
- net linesig31_{digital}: track 56.2 -> 55.9 mm, vias 2 -> 0
- net GND: vias 93 -> 94
Other:
- board text added: "+5V MOSI GND MISO SCK RST"
- board text added: "GND MOSI +5V RST SCK MISO"
