File: circuit/line-001-20260628/line-001-20260628.kicad_sch (KiCad schematic)
At the start: 217 parts, among them J1 Relay_{Power}, J2 Conn_{Signal}, J3 ICSP_{Arduino}, P1 USB-typeC, Q1 NJL7502L, Q10 NJL7502L, Q11 NJL7502L, Q12 NJL7502L, Q13 NJL7502L, Q14 NJL7502L, Q15 NJL7502L, Q16 NJL7502L, Q17 NJL7502L, Q18 NJL7502L, Q19 NJL7502L, Q2 NJL7502L, Q20 NJL7502L, Q21 NJL7502L, Q22 NJL7502L, Q23 NJL7502L, Q24 NJL7502L, Q25 NJL7502L, Q26 NJL7502L, Q27 NJL7502L, Q28 NJL7502L, Q29 NJL7502L, Q3 NJL7502L, Q30 NJL7502L, Q31 NJL7502L, Q32 NJL7502L, Q33 NJL7502L, Q34 NJL7502L, Q35 NJL7502L, Q36 NJL7502L, Q4 NJL7502L, Q5 NJL7502L, Q6 NJL7502L, Q7 NJL7502L, Q8 NJL7502L, Q9 NJL7502L, SW1 RESET, U1 LM339DR, U10 LM339DR, U11 LM339DR, U12 LM339DR, U13 LM339DR, U14 LM339DR, U15 LM339DR, U16 LM339DR, U17 ATmega2560-16A, U18 CH340G, U2 LM339DR, U3 LM339DR, U4 LM339DR, U5 LM339DR, U6 LM339DR, U7 LM339DR, U8 LM339DR, U9 LM339DR, Y1 16MHz, Y2 12MHz

Commit message: Update ラインセンサ基板のフットプリント紐づけを進めた
Parts:
- removed P1: USB-typeC, Connector_USB:USB_C_Receptacle_GCT_USB4105-xx-A_16P_TopMnt_Horizontal, symbol Connector:USB_C_Plug
- removed R82, R83: 22, Resistor_SMD:R_0805_2012Metric, symbol Device:R
- added D39: LED_{USB}, symbol Device:LED_Small
- added J4: USB_C_Receptacle_USB2.0_16P, symbol Connector:USB_C_Receptacle_USB2.0_16P
- added R82: 330, symbol Device:R_Small
- added R86: 5.1k, Resistor_SMD:R_0805_2012Metric, symbol Device:R
- added SW2: SW_SPDT, symbol Switch:SW_SPDT
Connections:
- net D+: now also J4.A6 (D+), J4.B6 (D+)
- net D-: now also J4.A7 (D-), J4.B7 (D-)
- net GND: now also D39.1 (K), J4.A1 (GND), J4.A12 (GND), J4.B1 (GND), J4.B12 (GND), J4.SH (SHIELD), R86.2
- net at R84.1: now also J4.A5 (CC1)
- new net: J4.B5 (CC2), R86.1
- new net: D39.2 (A), R82.2
- new net VBUS: J4.A4 (VBUS), J4.A9 (VBUS), J4.B4 (VBUS), J4.B9 (VBUS), R82.1
- no-connect marks 56 -> 43
Other:
- moved on the sheet: C29, C30, C31, C32, C33, J1, R81, R84, R85, U18, Y2

Commit message: Update ラインセンサ基板を更新
Parts:
- added D40, D41, D42, D43, D44, D45, D46, D47, D48, D49: LED, LED_THT:LED_D3.0mm, symbol Device:LED
- added D50: (no value), Package_TO_SOT_SMD:TSOT-23, symbol @Thrive_symbol_line:CH213K
- added Q37, Q38, Q39, Q40, Q41, Q42, Q43, Q44, Q45, Q46: NJL7502L, @Thrive_footprint_kicker:NJL7502L, symbol Device:Q_Photo_NPN_CE
- added R100, R83, R87, R88, R89, R90, R96, R97, R98, R99: 10k, Resistor_SMD:R_0805_2012Metric, symbol Device:R
- added R101, R102, R103, R104, R105, R91, R92, R93, R94, R95: 75, Resistor_SMD:R_0805_2012Metric, symbol Device:R
- D39: footprint (none) -> LED_SMD:LED_0603_1608Metric
- J4: footprint (none) -> Connector_USB:USB_C_Receptacle_HCTL_HC-TYPE-C-16P-01A
- R82: footprint (none) -> Resistor_SMD:R_0805_2012Metric
Connections:
- net +5V_{Line}: now also Q37.1 (C), Q38.1 (C), Q39.1 (C), Q40.1 (C), Q41.1 (C), Q42.1 (C), Q43.1 (C), Q44.1 (C), Q45.1 (C), Q46.1 (C), R101.2, R102.2, R103.2, R104.2, R105.2, R91.2, R92.2, R93.2, R94.2, R95.2
- net GND: now also D40.1 (K), D41.1 (K), D42.1 (K), D43.1 (K), D44.1 (K), D45.1 (K), D46.1 (K), D47.1 (K), D48.1 (K), D49.1 (K), D50.1 (GND), R100.1, R83.1, R87.1, R88.1, R89.1, R90.1, R96.1, R97.1, R98.1, R99.1
- net VBUS: now also SW2.3 (C), D50.2 (V_{O}); no longer J4.A4 (VBUS), J4.A9 (VBUS), J4.B4 (VBUS), J4.B9 (VBUS)
- net +5VD: now reaches SW2.2 (B)
- new net: D42.2 (A), R93.1
- new net: D48.2 (A), R104.1
- new net: D47.2 (A), R103.1
- new net: D41.2 (A), R92.1
- new net: Q42.2 (E), R96.2
- new net: Q44.2 (E), R98.2
- new net: D44.2 (A), R95.1
- new net: Q38.2 (E), R87.2
- new net: Q41.2 (E), R90.2
- new net: D40.2 (A), R91.1
- new net: D50.3 (V_{I}), J4.A4 (VBUS), J4.A9 (VBUS), J4.B4 (VBUS), J4.B9 (VBUS)
- new net: D49.2 (A), R105.1
- new net: D45.2 (A), R101.1
- new net: Q40.2 (E), R89.2
- new net: D46.2 (A), R102.1
- new net: D43.2 (A), R94.1
- new net: Q46.2 (E), R100.2
- new net: Q45.2 (E), R99.2
- new net: Q37.2 (E), R83.2
- new net: Q39.2 (E), R88.2
- new net: Q43.2 (E), R97.2
- no-connect marks 43 -> 44
Other:
- moved on the sheet: C24, C29, C30, C31, C32, C33, D37, D38, D39, J4, R79, R80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

Commit message: Update ラインセンサ基板の回路図とボード図を更新
Parts:
- removed D42, D43, D44, D47, D48, D49: LED, LED_THT:LED_D3.0mm, symbol Device:LED
- removed Q39, Q40, Q41, Q44, Q45, Q46: NJL7502L, @Thrive_footprint_kicker:NJL7502L, symbol Device:Q_Photo_NPN_CE
- removed R100, R88, R89, R90, R98, R99: 10k, Resistor_SMD:R_0805_2012Metric, symbol Device:R
- removed R103, R104, R105, R93, R94, R95: 75, Resistor_SMD:R_0805_2012Metric, symbol Device:R
- renumbered C25 to C24, C26 to C25, C27 to C26, C28 to C27, C24 to C28, D40 to D37, D41 to D38, D45 to D42, D46 to D43, D37 to D47, D38 to D48, D50 to D49, D39 to D50, R78 to R100, R81 to R101, R84 to R102, R86 to R103, R82 to R104, R85 to R105, R73 to R65, R74 to R66, R65 to R67, R66 to R68, R67 to R69, R68 to R70, R69 to R71, R70 to R72, R71 to R73, R72 to R74, R83 to R77, R87 to R78, R91 to R82, R92 to R83, R96 to R87, R97 to R88, R79 to R92, R80 to R93, R101 to R94, R102 to R95, R77 to R99
Connections:
- net +5VD: now also C1.2, C10.2, C11.2, C12.2, C13.2, C14.2, C15.2, C16.2, C2.2, C20.1, C23.1, C24.1, C25.1, C3.2, C32.2, C4.2, C5.2, C6.2, C7.2, C9.2, J3.2 (Pin_2), R65.1, U1.8 (V_{CC}), U10.8 (V_{CC}), U11.8 (V_{CC}), U12.8 (V_{CC}), U13.8 (V_{CC}), U14.8 (V_{CC}), U15.8 (V_{CC}), U16.8 (V_{CC}), U17.10 (VCC), U17.100 (AVCC), U17.31 (VCC), U17.61 (VCC), U17.80 (VCC), U18.16 (VCC), U2.8 (V_{CC}), U3.8 (V_{CC}), U4.8 (V_{CC}), U5.8 (V_{CC}), U6.8 (V_{CC}), U7.8 (V_{CC}), U9.8 (V_{CC})
- net +5V_{Line}: now also SW2.1 (A); no longer C1.2, C10.2, C11.2, C12.2, C13.2, C14.2, C15.2, C16.2, C2.2, C20.1, C23.1, C24.1, C25.1, C3.2, C32.2, C4.2, C5.2, C6.2, C7.2, C9.2, J3.2 (Pin_2), R65.1, U1.8 (V_{CC}), U10.8 (V_{CC}), U11.8 (V_{CC}), U12.8 (V_{CC}), U13.8 (V_{CC}), U14.8 (V_{CC}), U15.8 (V_{CC}), U16.8 (V_{CC}), U17.10 (VCC), U17.100 (AVCC), U17.31 (VCC), U17.61 (VCC), U17.80 (VCC), U18.16 (VCC), U2.8 (V_{CC}), U3.8 (V_{CC}), U4.8 (V_{CC}), U5.8 (V_{CC}), U6.8 (V_{CC}), U7.8 (V_{CC}), U9.8 (V_{CC})
- no-connect marks 44 -> 45
Other:
- moved on the sheet: D47, D48, R92, R93, SW2

Commit message: Update ラインセンサの部品配置を進めた
Parts:
- removed D1, D10, D11, D12, D13, D14, D15, D16, D17, D18, D19, D2, D20, D21, D22, D23, D24, D25, D26, D27, D28, D29, D3, D30, D31, D32, D33, D34, D35, D36, D37, D38, D4, D42, D43, D5, D6, D7, D8, D9: LED, LED_THT:LED_D3.0mm, symbol Device:LED
- removed Q42, Q43: NJL7502L, @Thrive_footprint_kicker:NJL7502L, symbol Device:Q_Photo_NPN_CE
- removed R1, R11, R12, R13, R14, R15, R2, R21, R22, R23, R24, R25, R3, R31, R32, R33, R34, R35, R4, R41, R42, R43, R44, R45, R5, R51, R52, R53, R54, R55, R61, R62, R67, R68, R69, R70, R77, R78, R87, R88: 10k, Resistor_SMD:R_0805_2012Metric, symbol Device:R
- removed R10, R16, R17, R18, R19, R20, R26, R27, R28, R29, R30, R36, R37, R38, R39, R40, R46, R47, R48, R49, R50, R56, R57, R58, R59, R6, R60, R63, R64, R7, R71, R72, R73, R74, R8, R82, R83, R9, R94, R95: 75, Resistor_SMD:R_0805_2012Metric, symbol Device:R
- added D1, D10, D11, D12, D13, D14, D15, D16, D17, D18, D19, D2, D20, D21, D22, D23, D24, D25, D26, D27, D28, D29, D3, D30, D31, D32, D33, D34, D35, D36, D37, D38, D39, D4, D40, D5, D6, D7, D8, D9: LED_Small, LED_THT:LED_D3.0mm, symbol Device:LED_Small
- added Q39, Q40: Q_Photo_NPN_CE, @Thrive_footprint_line:NJL7502L, symbol Device:Q_Photo_NPN_CE
- added R1, R10, R11, R12, R13, R14, R15, R16, R17, R18, R19, R2, R20, R21, R22, R23, R24, R25, R26, R27, R28, R29, R3, R30, R31, R32, R33, R34, R35, R36, R38, R4, R40, R41, R42, R43, R44, R45, R46, R47, R48, R49, R5, R50, R51, R52, R53, R54, R55, R56, R57, R58, R59, R6, R60, R61, R62, R63, R64, R65, R66, R67, R68, R69, R7, R70, R71, R72, R73, R74, R75, R76, R77, R78, R79, R8, R80, R9: R_Small, Resistor_SMD:R_0805_2012Metric, symbol Device:R_Small
- C1, C10, C11, C12, C13, C14, C15, C16, C2, C28, C3, C31, C33, C4, C5, C6, C7, C8, C9: value 100n -> C_Small
- C17, C19, C29, C30: value 22p -> C
- C18, C23, C24, C25, C32: value 100n -> C
- C20: value 470μ -> C
- C21, C22, C26, C27: value 10μ -> C
- D41: renamed from D47; value D40 -> LED_Small
- D42: renamed from D48; value D41 -> LED_Small
- D44: renamed from D50; value LED_{USB} -> LED_Small
- J1: value Relay_{Power} -> Conn_01x02_Pin
- J2: value Conn_{Signal} -> Conn_01x02_Pin
- J3: value ICSP_{Arduino} -> Conn_02x03_Odd_Even
- Q1, Q10, Q11, Q12, Q13, Q14, Q15, Q16, Q17, Q18, Q19, Q2, Q20, Q21, Q22, Q23, Q24, Q25, Q26, Q27, Q28, Q29, Q3, Q30, Q31, Q32, Q33, Q34, Q35, Q36, Q37, Q38, Q4, Q5, Q6, Q7, Q8, Q9: value NJL7502L -> Q_Photo_NPN_CE; footprint @Thrive_footprint_kicker:NJL7502L -> @Thrive_footprint_line:NJL7502L
- R81: renamed from R65; value 10k -> R
- R82: renamed from R66; value 1M -> R
- R83: renamed from R75; value 1k -> R
- R84: renamed from R76; value 1k -> R
- R85: renamed from R92; value 330 -> R_Small
- R86: renamed from R93; value 330 -> R_Small
- R87: renamed from R99; value 1k -> R
- R88: renamed from R100; value 1k -> R
- R89: renamed from R101; value 1M -> R
- R90: renamed from R102; value 5.1k -> R
- R91: renamed from R103; value 5.1k -> R
- R92: renamed from R104; value 330 -> R_Small
- R93: renamed from R105; value 10k -> R
- SW1: value RESET -> SW_Push
- SW2: footprint (none) -> @Thrive_footprint_line:SS12D01G4
- U1, U10, U11, U12, U13, U14, U15, U16, U2, U3, U4, U5, U6, U7, U8, U9: value LM339DR -> LM393DR; footprint Package_SO:SOIC-14_3.9x8.7mm_P1.27mm -> Package_SO:SOIC-8_3.9x4.9mm_P1.27mm
- Y1: value 16MHz -> Crystal
- Y2: value 12MHz -> Crystal
- renumbered D49 to D43
Connections:
- net +5VD: now also C8.2, U8.8 (V_{CC})
- net +5V_{Line}: now also Q39.1 (C), Q40.1 (C), R41.2, R42.2, R43.2, R44.2, R45.2, R46.2, R47.2, R48.2, R49.2, R50.2, R51.2, R52.2, R53.2, R54.2, R55.2, R56.2, R57.2, R58.2, R59.2, R60.2, R61.2, R62.2, R63.2, R64.2, R65.2, R66.2, R67.2, R68.2, R69.2, R70.2, R71.2, R72.2, R73.2, R74.2, R75.2, R76.2, R77.2, R78.2, R79.2, R80.2; no longer C8.2, U8.8 (V_{CC})
- net GND: now also D1.1 (K), D10.1 (K), D11.1 (K), D12.1 (K), D13.1 (K), D14.1 (K), D15.1 (K), D16.1 (K), D17.1 (K), D18.1 (K), D19.1 (K), D2.1 (K), D20.1 (K), D21.1 (K), D22.1 (K), D23.1 (K), D24.1 (K), D25.1 (K), D26.1 (K), D27.1 (K), D28.1 (K), D29.1 (K), D3.1 (K), D30.1 (K), D31.1 (K), D32.1 (K), D33.1 (K), D34.1 (K), D35.1 (K), D36.1 (K), D37.1 (K), D38.1 (K), D39.1 (K), D4.1 (K), D40.1 (K), D5.1 (K), D6.1 (K), D7.1 (K), D8.1 (K), D9.1 (K), R1.2, R10.2, R11.2, R12.2, R13.2, R14.2, R15.2, R16.2, R17.2, R18.2, R19.2, R2.2, R20.2, R21.2, R22.2, R23.2, R24.2, R25.2, R26.2, R27.2, R28.2, R29.2, R3.2, R30.2, R31.2, R32.2, R33.2, R34.2, R35.2, R36.2, R38.2, R4.2, R40.2, R5.2, R6.2, R7.2, R8.2, R9.2
- net linesig10_{digital}: now also U5.1 (1_{OUT}); no longer U5.7 (2_{OUT})
- net linesig10_{raw}: now also U5.3 (1_{IN+}), R10.1; no longer U5.5 (2_{IN+})
- net linesig11_{digital}: now also U6.7 (2_{OUT}); no longer U6.1 (1_{OUT})
- net linesig11_{raw}: now also U6.5 (2_{IN+}), R11.1; no longer U6.3 (1_{IN+})
- net linesig12_{digital}: now also U6.1 (1_{OUT}); no longer U6.7 (2_{OUT})
- net linesig12_{raw}: now also U6.3 (1_{IN+}), R12.1; no longer U6.5 (2_{IN+})
- net linesig13_{digital}: now also U7.7 (2_{OUT}); no longer U7.1 (1_{OUT})
- net linesig13_{raw}: now also U7.5 (2_{IN+}), R13.1; no longer U7.3 (1_{IN+})
- net linesig14_{digital}: now also U7.1 (1_{OUT}); no longer U7.7 (2_{OUT})
- net linesig14_{raw}: now also U7.3 (1_{IN+}), R14.1; no longer U7.5 (2_{IN+})
- net linesig15_{digital}: now also U8.7 (2_{OUT}); no longer U8.1 (1_{OUT})
- net linesig15_{raw}: now also U8.5 (2_{IN+}), R15.1; no longer U8.3 (1_{IN+})
- net linesig16_{digital}: now also U8.1 (1_{OUT}); no longer U8.7 (2_{OUT})
- net linesig16_{raw}: now also U8.3 (1_{IN+}), R16.1; no longer U8.5 (2_{IN+})
- net linesig17_{digital}: now also U9.7 (2_{OUT}); no longer U9.1 (1_{OUT})
- net linesig17_{raw}: now also U9.5 (2_{IN+}), R17.1; no longer U9.3 (1_{IN+})
- net linesig18_{digital}: now also U9.1 (1_{OUT}); no longer U9.7 (2_{OUT})
- net linesig18_{raw}: now also U9.3 (1_{IN+}), R18.1; no longer U9.5 (2_{IN+})
- net linesig19_{digital}: now also U10.7 (2_{OUT}); no longer U10.1 (1_{OUT})
- net linesig19_{raw}: now also U10.5 (2_{IN+}), R19.1; no longer U10.3 (1_{IN+})
- net linesig1_{digital}: now also U1.7 (2_{OUT}); no longer U1.1 (1_{OUT})
- net linesig1_{raw}: now also U1.5 (2_{IN+}), R1.1; no longer U1.3 (1_{IN+})
- net linesig20_{digital}: now also U10.1 (1_{OUT}); no longer U10.7 (2_{OUT})
- net linesig20_{raw}: now also U10.3 (1_{IN+}), R20.1; no longer U10.5 (2_{IN+})
- net linesig21_{digital}: now also U11.7 (2_{OUT}); no longer U11.1 (1_{OUT})
- net linesig21_{raw}: now also U11.5 (2_{IN+}), R21.1; no longer U11.3 (1_{IN+})
- net linesig22_{digital}: now also U11.1 (1_{OUT}); no longer U11.7 (2_{OUT})
- net linesig22_{raw}: now also U11.3 (1_{IN+}), R22.1; no longer U11.5 (2_{IN+})
- net linesig23_{digital}: now also U12.7 (2_{OUT}); no longer U12.1 (1_{OUT})
- net linesig23_{raw}: now also U12.5 (2_{IN+}), R23.1; no longer U12.3 (1_{IN+})
- net linesig24_{digital}: now also U12.1 (1_{OUT}); no longer U12.7 (2_{OUT})
- net linesig24_{raw}: now also U12.3 (1_{IN+}), R24.1; no longer U12.5 (2_{IN+})
- net linesig25_{digital}: now also U13.7 (2_{OUT}); no longer U13.1 (1_{OUT})
- net linesig25_{raw}: now also U13.5 (2_{IN+}), R25.1; no longer U13.3 (1_{IN+})
- net linesig26_{digital}: now also U13.1 (1_{OUT}); no longer U13.7 (2_{OUT})
- net linesig26_{raw}: now also U13.3 (1_{IN+}), R26.1; no longer U13.5 (2_{IN+})
- net linesig27_{digital}: now also U14.7 (2_{OUT}); no longer U14.1 (1_{OUT})
- net linesig27_{raw}: now also U14.5 (2_{IN+}), R27.1; no longer U14.3 (1_{IN+})
- net linesig28_{digital}: now also U14.1 (1_{OUT}); no longer U14.7 (2_{OUT})
- net linesig28_{raw}: now also U14.3 (1_{IN+}), R28.1; no longer U14.5 (2_{IN+})
- net linesig29_{digital}: now also U15.7 (2_{OUT}); no longer U15.1 (1_{OUT})
- net linesig29_{raw}: now also U15.5 (2_{IN+}), R29.1; no longer U15.3 (1_{IN+})
- net linesig2_{digital}: now also U1.1 (1_{OUT}); no longer U1.7 (2_{OUT})
- net linesig2_{raw}: now also U1.3 (1_{IN+}), R2.1; no longer U1.5 (2_{IN+})
- net linesig30_{digital}: now also U15.1 (1_{OUT}); no longer U15.7 (2_{OUT})
- net linesig30_{raw}: now also U15.3 (1_{IN+}), R30.1; no longer U15.5 (2_{IN+})
- net linesig31_{digital}: now also U16.7 (2_{OUT}); no longer U16.1 (1_{OUT})
- net linesig31_{raw}: now also U16.5 (2_{IN+}), R31.1; no longer U16.3 (1_{IN+})
- net linesig32_{digital}: now also U16.1 (1_{OUT}); no longer U16.7 (2_{OUT})
- net linesig32_{raw}: now also U16.3 (1_{IN+}), R32.1; no longer U16.5 (2_{IN+})
- net linesig33_{analog}: now also R33.1
- net linesig34_{analog}: now also R34.1
- net linesig35_{analog}: now also R35.1
- net linesig36_{analog}: now also R36.1
- net linesig3_{digital}: now also U2.7 (2_{OUT}); no longer U2.1 (1_{OUT})
- net linesig3_{raw}: now also U2.5 (2_{IN+}), R3.1; no longer U2.3 (1_{IN+})
- net linesig4_{digital}: now also U2.1 (1_{OUT}); no longer U2.7 (2_{OUT})
- net linesig4_{raw}: now also U2.3 (1_{IN+}), R4.1; no longer U2.5 (2_{IN+})
- net linesig5_{digital}: now also U3.7 (2_{OUT}); no longer U3.1 (1_{OUT})
- net linesig5_{raw}: now also U3.5 (2_{IN+}), R5.1; no longer U3.3 (1_{IN+})
- net linesig6_{digital}: now also U3.1 (1_{OUT}); no longer U3.7 (2_{OUT})
- net linesig6_{raw}: now also U3.3 (1_{IN+}), R6.1; no longer U3.5 (2_{IN+})
- net linesig7_{digital}: now also U4.7 (2_{OUT}); no longer U4.1 (1_{OUT})
- net linesig7_{raw}: now also U4.5 (2_{IN+}), R7.1; no longer U4.3 (1_{IN+})
- net linesig8_{digital}: now also U4.1 (1_{OUT}); no longer U4.7 (2_{OUT})
- net linesig8_{raw}: now also U4.3 (1_{IN+}), R8.1; no longer U4.5 (2_{IN+})
- net linesig9_{digital}: now also U5.7 (2_{OUT}); no longer U5.1 (1_{OUT})
- net linesig9_{raw}: now also U5.5 (2_{IN+}), R9.1; no longer U5.3 (1_{IN+})
- net linesig1^{side}_{raw}: now reaches Q38.2 (E)
- net linesig1^{side}_{raw}: now also Q37.2 (E), R38.1
- new net: D23.2 (A), R63.1
- new net: D19.2 (A), R59.1
- new net: D18.2 (A), R58.1
- new net: D35.2 (A), R75.1
- new net: D7.2 (A), R47.1
- new net: D34.2 (A), R74.1
- new net: D4.2 (A), R44.1
- new net: D21.2 (A), R61.1
- new net: D39.2 (A), R79.1
- new net: D14.2 (A), R54.1
- new net: D24.2 (A), R64.1
- new net: D37.2 (A), R77.1
- new net: D36.2 (A), R76.1
- new net: D8.2 (A), R48.1
- new net: D29.2 (A), R69.1
- new net: D1.2 (A), R41.1
- new net: D32.2 (A), R72.1
- new net: D40.2 (A), R80.1
- new net: D16.2 (A), R56.1
- new net: D10.2 (A), R50.1
- new net: D13.2 (A), R53.1
- new net: D31.2 (A), R71.1
- new net: D9.2 (A), R49.1
- new net: D30.2 (A), R70.1
- new net: D11.2 (A), R51.1
- new net: D3.2 (A), R43.1
- new net: D20.2 (A), R60.1
- new net: D22.2 (A), R62.1
- new net: D17.2 (A), R57.1
- new net: D28.2 (A), R68.1
- new net: D15.2 (A), R55.1
- new net: D12.2 (A), R52.1
- new net: D27.2 (A), R67.1
- new net: D26.2 (A), R66.1
- new net: D33.2 (A), R73.1
- new net: D5.2 (A), R45.1
- new net: D25.2 (A), R65.1
- new net: D38.2 (A), R78.1
- new net: D2.2 (A), R42.1
- new net: D6.2 (A), R46.1
- new net linesig2^{side}_{raw}: Q39.2 (E), Q40.2 (E), R40.1

Commit message: Update ラインセンサ基板の配線を進めた
Parts:
- removed C23, C24, C25: C, Capacitor_SMD:C_0805_2012Metric, symbol Device:C
- removed D33, D34, D35, D36: LED_Small, LED_THT:LED_D3.0mm, symbol Device:LED_Small
- removed Q33, Q34, Q35, Q36: Q_Photo_NPN_CE, @Thrive_footprint_line:NJL7502L, symbol Device:Q_Photo_NPN_CE
- removed R33, R34, R35, R36, R73, R74, R75, R76: R_Small, Resistor_SMD:R_0805_2012Metric, symbol Device:R_Small
- added C34, C35, C36, C37, C38: 100n, Capacitor_SMD:C_0805_2012Metric, symbol Device:C_Small
Connections:
- net +5VD: now also C34.1, C35.1, C36.1, C37.1, C38.1
- net GND: now also C34.2, C35.2, C36.2, C37.2, C38.2
- net LED1: no longer U17.52 (PG1)
- net LED2: no longer U17.51 (PG0)
- net linesig10_{digital}: now also U17.14 (PH2); no longer U17.63 (PJ0)
- net linesig11_{digital}: now also U17.91 (PF6); no longer U17.46 (PD3)
- net linesig12_{digital}: now also U17.90 (PF7); no longer U17.45 (PD2)
- net linesig13_{digital}: now also U17.77 (PA1); no longer U17.44 (PD1)
- net linesig14_{digital}: now also U17.76 (PA2); no longer U17.43 (PD0)
- net linesig15_{digital}: now also U17.75 (PA3); no longer U17.78 (PA0)
- net linesig16_{digital}: now also U17.74 (PA4); no longer U17.77 (PA1)
- net linesig17_{digital}: now also U17.67 (PJ4); no longer U17.76 (PA2)
- net linesig18_{digital}: now also U17.66 (PJ3); no longer U17.75 (PA3)
- net linesig19_{digital}: now also U17.58 (PC5); no longer U17.74 (PA4)
- net linesig1_{digital}: now also U17.26 (PB7); no longer U17.15 (PH3)
- net linesig20_{digital}: now also U17.57 (PC4); no longer U17.73 (PA5)
- net linesig21_{digital}: now also U17.56 (PC3); no longer U17.72 (PA6)
- net linesig22_{digital}: now also U17.55 (PC2); no longer U17.71 (PA7)
- net linesig23_{digital}: now also U17.54 (PC1); no longer U17.60 (PC7)
- net linesig24_{digital}: now also U17.53 (PC0); no longer U17.59 (PC6)
- net linesig25_{digital}: now also U17.52 (PG1); no longer U17.58 (PC5)
- net linesig26_{digital}: now also U17.51 (PG0); no longer U17.57 (PC4)
- net linesig27_{digital}: now also U17.38 (PL3); no longer U17.56 (PC3)
- net linesig28_{digital}: now also U17.37 (PL2); no longer U17.55 (PC2)
- net linesig29_{digital}: now also U17.36 (PL1); no longer U17.54 (PC1)
- net linesig2_{digital}: now also U17.25 (PB6); no longer U17.16 (PH4)
- net linesig30_{digital}: now also U17.35 (PL0); no longer U17.53 (PC0)
- net linesig31_{digital}: now also U17.28 (PG3); no longer U17.50 (PD7)
- net linesig32_{digital}: now also U17.27 (PH7); no longer U17.70 (PG2)
- net linesig3_{digital}: now also U17.24 (PB5); no longer U17.17 (PH5)
- net linesig4_{digital}: now also U17.23 (PB4); no longer U17.18 (PH6)
- net linesig5_{digital}: now also U17.19 (PB0); no longer U17.23 (PB4)
- net linesig6_{digital}: now also U17.18 (PH6); no longer U17.24 (PB5)
- net linesig7_{digital}: now also U17.17 (PH5); no longer U17.25 (PB6)
- net linesig8_{digital}: now also U17.16 (PH4); no longer U17.26 (PB7)
- net linesig9_{digital}: now also U17.15 (PH3); no longer U17.64 (PJ1)
- net linesig33_{analog}: no longer names the net of U17.97 (PF0)
- net linesig34_{analog}: no longer names the net of U17.96 (PF1)
- net linesig35_{analog}: no longer names the net of U17.95 (PF2)
- net linesig36_{analog}: no longer names the net of U17.94 (PF3)
- no-connect marks 45 -> 51
Other:
- moved on the sheet: C20, C28

Commit message: Update ラインセンサ基板を進めた、GND孤立がひどい
Parts:
- C1, C10, C11, C12, C13, C14, C15, C16, C2, C28, C3, C33, C4, C5, C6, C7, C8, C9: value C_Small -> 100n
- C17, C19, C29, C30: value C -> 22p; footprint Capacitor_SMD:C_0805_2012Metric -> Capacitor_SMD:C_0603_1608Metric
- C18, C32: value C -> 100n
- C20: value C -> 100μ; footprint Capacitor_SMD:C_0805_2012Metric -> Capacitor_SMD:C_1206_3216Metric
- D41: value LED_Small -> LED1
- D42: value LED_Small -> LED2
- D44: value LED_Small -> USB
- R1, R10, R11, R12, R13, R14, R15, R16, R17, R18, R19, R2, R20, R21, R22, R23, R24, R25, R26, R27, R28, R29, R3, R30, R31, R32, R38, R4, R40, R5, R6, R7, R8, R9: value R_Small -> 10k
- R41, R42, R43, R44, R45, R46, R47, R48, R49, R50, R51, R52, R53, R54, R55, R56, R57, R58, R59, R60, R61, R62, R63, R64, R65, R66, R67, R68, R69, R70, R71, R72, R77, R78, R79, R80: value R_Small -> 75
- R81: value R -> 10k
- R82, R89: value R -> 1M
- R85, R86, R92: value R_Small -> 330
- R90, R91: value R -> 5.1k
- R93: value R -> 4.7k
- Y1: value Crystal -> 16MHz; footprint Crystal:Crystal_HC49-4H_Vertical -> Crystal:Crystal_SMD_SeikoEpson_FA238-4Pin_3.2x2.5mm
- Y2: value Crystal -> 12MHz; footprint Crystal:Crystal_HC49-4H_Vertical -> Crystal:Crystal_SMD_SeikoEpson_FA238V-4Pin_3.2x2.5mm
Connections:
- net XTAL1: now also Y1.3; no longer Y1.2
- net at C29.2, R89.1, U18.7 (XI): now also Y2.3; no longer Y2.2
Other:
- moved on the sheet: C20

Commit message: Update ラインセンサ基板のPCBを進めた
Other:
- moved on the sheet: C28, U17
