File: circuit/neopixel-001-20260528/neopixel-001-20260528.kicad_sch (KiCad schematic)
At the start: 71 parts, among them J1 Conn_Sub, J2 Conn_01x02_Pin, J3 Conn_01x02_Pin, P1 ESP32C3_{1}, P10 unitV3, P11 unitV4, P12 unitV4, P2 ESP32C3_{1}, P3 ESP32C3_{2}, P4 ESP32C3_{2}, P5 unitV1, P6 unitV1, P7 unitV2, P8 unitV2, P9 unitV3, Q1 NMOS, Q2 NMOS, Q3 NMOS, SW1 SW_SPST_LED, SW2 SW_SPST_LED, SW4 SW_SPST_LED, U1 SSD1306, U2 Aexit_0-50_Voltmeter, U3 74AHC1G04, U4 74AHC1G04, U5 74AHC1G04

Commit message: Update NeoPixel基板をプッシュした
Parts:
- Q1, Q2, Q3: value NMOS -> BSS138
Changed lines of the file:
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@@
 			)
 		)
-		(property "Value" "NMOS"
+		(property "Value" "BSS138"
 			(at 335.28 77.47 0)
 			(show_name no)
@@
 			)
 		)
-		(property "Value" "NMOS"
+		(property "Value" "BSS138"
 			(at 335.28 110.49 0)
 			(show_name no)
@@
 			)
 		)
-		(property "Value" "NMOS"
+		(property "Value" "BSS138"
 			(at 335.28 44.45 0)
 			(show_name no)
